File: Flotelli/Flotelli.sch (EAGLE design)
At the start: 64 parts, among them J1 FTDI-SER-6-PP, J3 DF12-32-DP, J4 DF12-60-DP, U3 STM32F429-LQFP144, Y1-C1 22pF, Y1-C2 22pF, Y1-R1 390R

Commit message: Update Flotelli
Parts:
- C1, C10, C11, C12, C13, C14, C15, C16, C17, C18, C2, C3, C4, C5, C6, C7, C8, C9, Y1-C1, Y1-C2: device ell-i:C0402 -> ELL-i-Passives:C0402
- D2: device ell-i:LED0603 -> SparkFun-LED:LED-GREEN0603
- J3: value DF12-32-DP -> DF12-32DP-0.5V; device ell-i:DF12-32-DP -> ELL-i-Connectors:DF12-32DP-0.5V
- J4: value DF12-60-DP -> DF12-60DP; device ell-i:DF12-60-DP -> ELL-i-Connectors:DF12-60DP
- R1, R2, R33, Y1-R1: device ell-i:R0402 -> ELL-i-Passives:R0402
- SV2, SV3, SV4, SV5: value (none) -> M09LOCK; device con-lstb:MA09-1 -> SparkFun-Connectors:M09LOCK
- U1: device ell-i:LAN8720-H -> ELL-i-DigitalIC:LAN8720-H
- U3: value STM32F429-LQFP144 -> STM32F429ZIT; device ell-i:STM32F429-LQFP144 -> ELL-i-DigitalIC:STM32F429ZIT
Connections:
- net IO5: now also U3PA.PA13-SWDIO; no longer U3PA.PA13
- net TX2: now also U3PA.PA14-SWCLK; no longer U3PA.PA14
Other:
- moved on the sheet: U3PA
Changed lines of the file:
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@@
 <?xml version="1.0" encoding="utf-8"?>
 <!DOCTYPE eagle SYSTEM "eagle.dtd">
-<eagle version="6.5.0">
+<eagle version="6.4">
 <drawing>
 <settings>
@@
 </classes>
 <parts>
-<part name="C1" library="ell-i" deviceset="C" device="0402" value="33n"/>
-<part name="C6" library="ell-i" deviceset="C" device="0402" value="100nF"/>
-<part name="C7" library="ell-i" deviceset="C" device="0402" value="1uF"/>
-<part name="C8" library="ell-i" deviceset="C" device="0402" value="1uF"/>
-<part name="C9" library="ell-i" deviceset="C" device="0402" value="100nF"/>
-<part name="D2" library="ell-i" deviceset="LED0603" device="" value="GRN"/>
-<part name="R1" library="ell-i" deviceset="R" device="0402" value="150R"/>
-<part name="R33" library="ell-i" deviceset="R" device="0402" value="1k5"/>
+<part name="C1" library="ELL-i-Passives" deviceset="C" device="0402" value="33n"/>
+<part name="C6" library="ELL-i-Passives" deviceset="C" device="0402" value="100nF"/>
+<part name="C7" library="ELL-i-Passives" deviceset="C" device="0402" value="1uF"/>
+<part name="C8" library="ELL-i-Passives" deviceset="C" device="0402" value="1uF"/>
+<part name="C9" library="ELL-i-Passives" deviceset="C" device="0402" value="100nF"/>
+<part name="D2" library="SparkFun-LED" deviceset="LED-GREEN" device="0603" value="GRN"/>
+<part name="R1" library="ELL-i-Passives" deviceset="R" device="0402" value="150R"/>
+<part name="R33" library="ELL-i-Passives" deviceset="R" device="0402" value="1k5"/>
 <part name="GNDI3" library="supply1" deviceset="GNDI" device=""/>
 <part name="+3V7" library="supply1" deviceset="+3V3" device=""/>
@@
 <part name="PC15" library="testpad" deviceset="TPS" device="B1,27"/>
 <part name="PC12" library="testpad" deviceset="TPS" device="B1,27"/>
-<part name="Y1-C1" library="ell-i" deviceset="C" device="0402" value="22pF"/>
-<part name="Y1-C2" library="ell-i" deviceset="C" device="0402" value="22pF"/>
-<part name="Y1-R1" library="ell-i" deviceset="R" device="0402" value="390R"/>
+<part name="Y1-C1" library="ELL-i-Passives" deviceset="C" device="0402" value="22pF"/>
+<part name="Y1-C2" library="ELL-i-Passives" deviceset="C" device="0402" value="22pF"/>
+<part name="Y1-R1" library="ELL-i-Passives" deviceset="R" device="0402" value="390R"/>
 <part name="GNDI8" library="supply1" deviceset="GNDI" device=""/>
 <part name="Y1" library="crystal" deviceset="CRYSTAL" device="SM49"/>
-<part name="C2" library="ell-i" deviceset="C" device="0402" value="1uF"/>
-<part name="C3" library="ell-i" deviceset="C" device="0402" value="10nF"/>
+<part name="C2" library="ELL-i-Passives" deviceset="C" device="0402" value="1uF"/>
+<part name="C3" library="ELL-i-Passives" deviceset="C" device="0402" value="10nF"/>
 <part name="FB2" library="ell-i" deviceset="LQM15" device="" value="BLM15A"/>
 <part name="FB1" library="ell-i" deviceset="LQM15" device="" value="BLM15A"/>
@@
 <part name="GNDI25" library="supply1" deviceset="GNDI" device=""/>
 <part name="U$1" library="alo" deviceset="FR-A4L" device=""/>
-<part name="U1" library="ell-i" deviceset="LAN8720" device="-H"/>
+<part name="U1" library="ELL-i-DigitalIC" deviceset="LAN8720" device="-H"/>
 <part name="GNDI2" library="supply1" deviceset="GNDI" device=""/>
-<part name="C4" library="ell-i" deviceset="C" device="0402" value="2.2uF"/>
-<part name="C5" library="ell-i" deviceset="C" device="0402" value="2.2uF"/>
+<part name="C4" library="ELL-i-Passives" deviceset="C" device="0402" value="2.2uF"/>
+<part name="C5" library="ELL-i-Passives" deviceset="C" device="0402" value="2.2uF"/>
 <part name="GNDI4" library="supply1" deviceset="GNDI" device=""/>
 <part name="GNDI9" library="supply1" deviceset="GNDI" device=""/>
-<part name="U3" library="ell-i" deviceset="STM32F429-LQFP144" device=""/>
-<part name="SV2" library="con-lstb" deviceset="MA09-1" device=""/>
-<part name="SV3" library="con-lstb" deviceset="MA09-1" device=""/>
-<part name="SV4" library="con-lstb" deviceset="MA09-1" device=""/>
-<part name="SV5" library="con-lstb" deviceset="MA09-1" device=""/>
+<part name="U3" library="ELL-i-DigitalIC" deviceset="STM32F429Z" device="T" technology="I" value="STM32F429ZIT"/>
+<part name="SV2" library="SparkFun-Connectors" deviceset="M09" device="LOCK"/>
+<part name="SV3" library="SparkFun-Connectors" deviceset="M09" device="LOCK"/>
+<part name="SV4" library="SparkFun-Connectors" deviceset="M09" device="LOCK" value="M09LOCK"/>
+<part name="SV5" library="SparkFun-Connectors" deviceset="M09" device="LOCK"/>
 <part name="SV6" library="con-lsta" deviceset="FE06W" device=""/>
-<part name="C10" library="ell-i" deviceset="C" device="0402" value="100nF"/>
-<part name="C11" library="ell-i" deviceset="C" device="0402" value="100nF"/>
-<part name="C12" library="ell-i" deviceset="C" device="0402" value="100nF"/>
-<part name="C13" library="ell-i" deviceset="C" device="0402" value="100nF"/>
-<part name="C14" library="ell-i" deviceset="C" device="0402" value="100nF"/>
-<part name="C15" library="ell-i" deviceset="C" device="0402" value="100nF"/>
-<part name="C16" library="ell-i" deviceset="C" device="0402" value="100nF"/>
-<part name="C17" library="ell-i" deviceset="C" device="0402" value="100nF"/>
-<part name="C18" library="ell-i" deviceset="C" device="0402" value="100nF"/>
+<part name="C10" library="ELL-i-Passives" deviceset="C" device="0402" value="100nF"/>
+<part name="C11" library="ELL-i-Passives" deviceset="C" device="0402" value="100nF"/>
+<part name="C12" library="ELL-i-Passives" deviceset="C" device="0402" value="100nF"/>
+<part name="C13" library="ELL-i-Passives" deviceset="C" device="0402" value="100nF"/>
+<part name="C14" library="ELL-i-Passives" deviceset="C" device="0402" value="100nF"/>
+<part name="C15" library="ELL-i-Passives" deviceset="C" device="0402" value="100nF"/>
+<part name="C16" library="ELL-i-Passives" deviceset="C" device="0402" value="100nF"/>
+<part name="C17" library="ELL-i-Passives" deviceset="C" device="0402" value="100nF"/>
+<part name="C18" library="ELL-i-Passives" deviceset="C" device="0402" value="100nF"/>
 <part name="VIA1" library="ell-i" deviceset="VIA" device="-0.3"/>
 <part name="VIA2" library="ell-i" deviceset="VIA" device="-0.3"/>
@@
 <part name="D3" library="ell-i" deviceset="BAT60J" device=""/>
 <part name="+3V1" library="supply1" deviceset="+3V3" device=""/>
-<part name="R2" library="ell-i" deviceset="R" device="0402" value="10k"/>
+<part name="R2" library="ELL-i-Passives" deviceset="R" device="0402" value="10k"/>
 <part name="GNDI1" library="supply1" deviceset="GNDI" device=""/>
-<part name="J3" library="ell-i" deviceset="DF12-32-DP" device=""/>
+<part name="J3" library="ELL-i-Connectors" deviceset="DF12-32DP-0.5V" device=""/>
 <part name="FID1" library="microbuilder" deviceset="FIDUCIAL" device="1X2.5" value="FIDUCIAL1X2.5"/>
 <part name="FID2" library="microbuilder" deviceset="FIDUCIAL" device="&quot;&quot;"/>
 <part name="FID3" library="microbuilder" deviceset="FIDUCIAL" device="&quot;&quot;"/>
 <part name="FID4" library="microbuilder" deviceset="FIDUCIAL" device="&quot;&quot;"/>
-<part name="J4" library="ell-i" deviceset="DF12-60-DP" device=""/>
+<part name="J4" library="ELL-i-Connectors" deviceset="DF12-60DP" device=""/>
 </parts>
 <sheets>
@@
 <attribute name="VALUE" x="33.02" y="104.14" size="1.778" layer="96"/>
 </instance>
-<instance part="D2" gate="G$1" x="30.48" y="162.56" rot="R270"/>
+<instance part="D2" gate="G$1" x="30.48" y="162.56"/>
 <instance part="R1" gate="G$1" x="30.48" y="152.4" rot="R270"/>
 <instance part="R33" gate="G$1" x="38.1" y="83.82" rot="R90"/>
@@
 <instance part="U3" gate="PF" x="289.56" y="149.86"/>
 <instance part="U3" gate="PG" x="289.56" y="101.6"/>
-<instance part="SV2" gate="1" x="307.34" y="157.48"/>
-<instance part="SV3" gate="1" x="307.34" y="127"/>
-<instance part="SV4" gate="1" x="307.34" y="96.52"/>
-<instance part="SV5" gate="1" x="307.34" y="68.58"/>
+<instance part="SV2" gate="G$1" x="307.34" y="157.48"/>
+<instance part="SV3" gate="G$1" x="307.34" y="127"/>
+<instance part="SV4" gate="G$1" x="307.34" y="96.52"/>
+<instance part="SV5" gate="G$1" x="307.34" y="68.58"/>
 <instance part="D3" gate="G$1" x="43.18" y="109.22" smashed="yes" rot="R90">
 <attribute name="NAME" x="37.338" y="108.204" size="1.778" layer="95"/>
@@
 <wire x1="248.92" y1="68.58" x2="261.62" y2="68.58" width="0.1524" layer="91"/>
 <label x="261.62" y="68.58" size="1.016" layer="95" xref="yes"/>
-<pinref part="U3" gate="PA" pin="PA13"/>
+<pinref part="U3" gate="PA" pin="PA13-SWDIO"/>
 </segment>
 </net>
@@
 <pinref part="D2" gate="G$1" pin="C"/>
 <pinref part="R1" gate="G$1" pin="1"/>
-<wire x1="30.48" y1="160.02" x2="30.48" y2="157.48" width="0.1524" layer="91"/>
 </segment>
 </net>
@@
 <wire x1="261.62" y1="66.04" x2="248.92" y2="66.04" width="0.1524" layer="91"/>
 <label x="261.62" y="66.04" size="1.016" layer="95" xref="yes"/>
-<pinref part="U3" gate="PA" pin="PA14"/>
+<pinref part="U3" gate="PA" pin="PA14-SWCLK"/>
 </segment>
 </net>
@@
 <pinref part="+3V7" gate="G$1" pin="+3V3"/>
 <pinref part="D2" gate="G$1" pin="A"/>
-<wire x1="30.48" y1="170.18" x2="30.48" y2="167.64" width="0.1524" layer="91"/>
-</segment>
-<segment>
+<wire x1="30.48" y1="170.18" x2="30.48" y2="165.1" width="0.1524" layer="91"/>
+</segment>
+<segment>

Commit message: Replaced FTDI header with a new one
Parts:
- J1: device ell-i:FTDI-SER-6-PP -> ELL-i-Connectors:FTDI-SER-6-PP
Changed lines of the file:
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@@
 <part name="GNDI21" library="supply1" deviceset="GNDI" device=""/>
 <part name="U$2" library="alo" deviceset="FR-A4L" device=""/>
-<part name="J1" library="ell-i" deviceset="FTDI-SER-6" device="-PP" value="FTDI-SER-6-PP"/>
+<part name="J1" library="ELL-i-Connectors" deviceset="FTDI-SER-6" device="-PP" value="FTDI-SER-6-PP"/>
 <part name="+5V1" library="tinycircuits" deviceset="+5V" device="" value="+5V"/>
 <part name="VCC1" library="tinycircuits" deviceset="VCC" device="" value="VCC"/>

Commit message: Replaces the 6-pin female header on Flotelli
Parts:
- SV6: device con-lsta:FE06W -> ELL-i-Connectors:M06
Changed lines of the file:
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@@
 <?xml version="1.0" encoding="utf-8"?>
 <!DOCTYPE eagle SYSTEM "eagle.dtd">
-<eagle version="6.4">
+<eagle version="6.5.0">
 <drawing>
 <settings>
@@
 <part name="SV4" library="SparkFun-Connectors" deviceset="M09" device="LOCK" value="M09LOCK"/>
 <part name="SV5" library="SparkFun-Connectors" deviceset="M09" device="LOCK"/>
-<part name="SV6" library="con-lsta" deviceset="FE06W" device=""/>
+<part name="SV6" library="ELL-i-Connectors" deviceset="M06" device=""/>
 <part name="C10" library="ELL-i-Passives" deviceset="C" device="0402" value="100nF"/>
 <part name="C11" library="ELL-i-Passives" deviceset="C" device="0402" value="100nF"/>

Commit message: Flotelli pins defined per the latest pin order table.
There are still some errors in the table.  We will fix them next.

Also has Flotelli brd, very preliminary.
Parts:
- removed PC12: TPSB1,27, testpad:TPSB1,27
- removed SV6: (no value), ELL-i-Connectors:M06
- removed U3: STM32F429ZIT, ELL-i-DigitalIC:STM32F429ZIT
- added BR00, BR01, BR02, BR03, BR04, BR05, BR06, BR07, BR08, BR09, BR10, BR11, BR12, BR13, BR14, BR15, BR16, BR17, BR18, BR19, BR20, BR21, BR22, BR23, BR24, BR25, BR26, BR27, BR28, BR29, BR30, BR31: 100, ELL-i-Passives:R0603
- added CSSPIN: TPSB1,27, testpad:TPSB1,27
- added J2: DF12-ELLI-RECEPTABLE-BOTTOM, ELL-i-Connectors:DF12-ELLI-RECEPTABLE-BOTTOM
- added U2: LCMXO2-2000HC-4TG144, ELL-i-DigitalIC:LCMXO2-2000HC-4TG144
- added U4: (no value), ELL-i-DigitalIC:LAN8720-H
- added X1, X2, X3, X4: M-BOLT-2, ELL-i-Connectors:M-BOLT-2
- FID1: value FIDUCIAL1X2.5 -> FIDUCIAL""; device microbuilder:FIDUCIAL1X2.5 -> microbuilder:FIDUCIAL""
- J4: value DF12-60DP -> DF12-ELLI-HEADER-TOP; device ELL-i-Connectors:DF12-60DP -> ELL-i-Connectors:DF12-ELLI-HEADER-TOP
- U1: value (none) -> STM32F429ZIT; device ELL-i-DigitalIC:LAN8720-H -> ELL-i-DigitalIC:STM32F429ZIT
Connections:
- removed net AD0: J3.11, U3PA.PA0-ADC_IN0
- removed net AD1-ETH_REF_CLK: J3.9, U1.NINT/REFCLKO, U3PA.PA1-ADC_IN1
- removed net AD10: U3PC.PC0-ADC_IN10
- removed net AD11-ETH_MDC: U1.MDC, U3PC.PC1-ADC_IN11
- removed net AD12: U3PC.PC2-ADC_IN12
- removed net AD13: U3PC.PC3-ADC_IN13
- removed net AD14-ETH_RXD0: U1.RXD0, U3PC.PC4-ADC_IN14
- removed net AD15-ETH_RXD1: U1.RXD1, U3PC.PC5-ADC_IN15
- removed net AD2-ETH_MDIO: J3.7, U1.MDIO, U3PA.PA2-ADC_IN2
- removed net AD3: J3.5, U3PA.PA3-ADC_IN3
- removed net AD4: J3.3, U3PA.PA4-ADC_IN4
- removed net AD5: J3.1, U3PA.PA5-ADC_IN5
- removed net AD6: U3PA.PA6-ADC_IN6
- removed net AD7-ETH_CRSDV: U1.CRS_DV, U3PA.PA7-ADC_IN7
- removed net AD8: U3PB.PB0-ADC_IN8
- removed net AD9: U3PB.PB1-ADC_IN9
- removed net ETH_TEX_EN: U1.TXEN, U3PB.PB11
- removed net IO0: J3.24, U3PA.PA8
- removed net IO1: J3.26, U3PA.PA9
- removed net IO2: J3.28, U3PA.PA10
- removed net IO3: J3.30, U3PA.PA11, U3PC.PC9
- removed net IO4: J3.32, U3PA.PA12, U3PC.PC8
- removed net IO5: J3.31, U3PA.PA13-SWDIO
- removed net IO8: J3.25, U3PB.PB10
- removed net MISO1: U3PB.PB4
- removed net MISO_ETH: U3PB.PB14
- removed net MOSI1: U3PB.PB5
- removed net MOSI_ETH: U3PB.PB15
- removed net N$1: U3PB.PB2
- removed net N$9: PC12.PP, U3PC.PC12
- removed net PB6: U3PB.PB6
- removed net PB7: U3PB.PB7
- removed net PD2: U3PD.PD2
- removed net PF2: J4.13, U3PF.PF2
- removed net RX2: R2.2, U3PA.PA15
- removed net SCK1: U3PB.PB3
- removed net SCL1: U3PB.PB8
- removed net SDA1: U3PB.PB9
- removed net SPR1: U3PC.PC6
- removed net SPR2: U3PC.PC7
- removed net TX2: J1.RXD, U3PA.PA14-SWCLK
- new net A0: J3.11, U1PA.PA0-ADC_IN0
- new net A1: U1PF.PF6
- new net A2: J3.3, U1PA.PA4-ADC_IN4
- new net A3: J3.1, U1PA.PA5-ADC_IN5
- new net A4: U1PB.PB9
- new net A5: U1PB.PB6
- new net CSSPIN: CSSPIN.PP, U1PC.PC12
- new net D0: J3.28, U1PA.PA10
- new net D1: J3.26, U1PA.PA9
- new net D10: R2.2, U1PA.PA15
- new net D11: U1PB.PB5
- new net D12: U1PA.PA6-ADC_IN6
- new net D13: U1PB.PB3
- new net D2: U1PD.PD2
- new net D5: U1PB.PB1-ADC_IN9
- new net D6: J3.5, U1PA.PA3-ADC_IN3
- new net D7: U1PB.PB8
- new net D8: U1PG.PG6
- new net D9: U1PB.PB0-ADC_IN8
- new net E0: U1PF.PF7
- new net E1: U1PF.PF8
- new net E10: U1PC.PC6
- new net E11: U1PC.PC7
- new net E12: U1PB.PB11
- new net E13: J3.25, U1PB.PB10
- new net E14: U1PB.PB12
- new net E15: U1PB.PB15
- new net E16: U1PB.PB14
- new net E17: U1PB.PB13
- new net E18: U1PC.PC11
- new net E19: U1PC.PC10
- new net E2: U1PF.PF9
- new net E3: U1PF.PF10
- new net E8: U1PG.PG7
- new net ETH_CLK: J3.9, U1PA.PA1-ADC_IN1, U4.NINT/REFCLKO
- new net ETH_CRS: U1PA.PA7-ADC_IN7, U4.CRS_DV
- new net ETH_MDC: U1PC.PC1-ADC_IN11, U4.MDC
- new net ETH_MDIO: J3.7, U1PA.PA2-ADC_IN2, U4.MDIO
- new net ETH_RXD0: U1PC.PC4-ADC_IN14, U4.RXD0
- new net ETH_RXD1: U1PC.PC5-ADC_IN15, U4.RXD1
- new net ETH_TXEN: U1PG.PG11, U4.TXEN
- new net FPGA_SN: U1PB.PB2
- new net JTCK: J1.RXD, U1PA.PA14-SWCLK
- new net JTDI: J3.30, U1PA.PA11, U1PC.PC9
- new net JTMS: J3.31, U1PA.PA13-SWDIO
- new net JTRST: U1PB.PB4
- new net MCO: J3.24, U1PA.PA8
- new net MEM_A0: U1PF.PF0
- new net MEM_A1: U1PF.PF1
- new net MEM_A10: U1PG.PG0, U1PG.PG1
- new net MEM_A12: U1PG.PG2
- new net MEM_A13: U1PG.PG3
- new net MEM_A14: U1PG.PG4
- new net MEM_A15: U1PG.PG5
- new net MEM_A16: U1PD.PD11, U2MACHXO2-CSBGA132-640-LEFT.PL_/5C/5C/9A/13A
- new net MEM_A17: U1PD.PD12, U2MACHXO2-CSBGA132-640-LEFT.PL_/5D/5D/9B/13B
- new net MEM_A18: U1PD.PD13, U2MACHXO2-CSBGA132-256-LEFT.PL_5A/6A/8A/10A/14A
- new net MEM_A19: U1PE.PE3, U2MACHXO2-CSBGA132-256-LEFT.PL_5B/6B/8B/10B/14B
- new net MEM_A2: U1PF.PF2
- new net MEM_A20: U1PE.PE4
- new net MEM_A21: U1PE.PE5, U2MACHXO2-CSBGA132-640-BOTTOM.PB_/4C/6A/6A/7A
- new net MEM_A22: U1PE.PE6, U2MACHXO2-CSBGA132-256-BOTTOM.PB_7C/12C/18A/21A/24A
- new net MEM_A23: U1PE.PE2, U2MACHXO2-CSBGA132-256-BOTTOM.PB_7D/12D/18B/21B/24B
- new net MEM_A3: U1PF.PF3
- new net MEM_A4: U1PF.PF4
- new net MEM_A5: U1PF.PF5
- new net MEM_A6: U1PF.PF12
- new net MEM_A7: U1PF.PF13
- new net MEM_A8: U1PF.PF14
- new net MEM_A9: U1PF.PF15
- new net MEM_CLK: U1PD.PD3
- new net MEM_CS1: U1PD.PD7, U2MACHXO2-QFN32-256.PB_4B/6D/9B/11B/13B
- new net MEM_CS2: U1PG.PG9
- new net MEM_CS3: U1PG.PG10
- new net MEM_CS4: U1PG.PG12
- new net MEM_D0: U1PD.PD14, U2MACHXO2-CSBGA132-1200-LEFT.PL_//2A/1A/3A
- new net MEM_D1: U1PD.PD15, U2MACHXO2-CSBGA132-1200-LEFT.PL_//2B/1B/3B
- new net MEM_D10: U1PE.PE13, U2MACHXO2-CSBGA132-1200-LEFT.PL_//4C/6A/9A
- new net MEM_D11: U1PE.PE14, U2MACHXO2-CSBGA132-1200-LEFT.PL_//4D/6B/9B
- new net MEM_D12: U1PE.PE15, U2MACHXO2-TEFQ144-2000.PL_///7A/10A/10A
- new net MEM_D13: U1PD.PD8, U2MACHXO2-TEFQ144-2000.PL_///7B/10B/10B
- new net MEM_D14: U1PD.PD9, U2MACHXO2-CSBGA132-256-LEFT.PL_3C/5A/5A/7C/10C
- new net MEM_D15: U1PD.PD10, U2MACHXO2-CSBGA132-256-LEFT.PL_3D/5B/5B/7D/10D
- new net MEM_D2: U1PD.PD0, U2MACHXO2-CSBGA132-256-LEFT.PL_2A/2A/2C/2A/4A
- new net MEM_D3: U1PD.PD1, U2MACHXO2-CSBGA132-256-LEFT.PL_2B/2B/2D/2B/4B
- new net MEM_D4: U1PE.PE7, U2MACHXO2-CSBGA132-256-LEFT.PL_2C/2C/3A/3A/6A
- new net MEM_D5: U1PE.PE8, U2MACHXO2-CSBGA132-256-LEFT.PL_2D/2D/3B/3B/6B
- new net MEM_D6: U1PE.PE9, U2MACHXO2-CSBGA132-256-LEFT.PL_3A/3A/3C/4A/7A
- new net MEM_D7: U1PE.PE10, U2MACHXO2-CSBGA132-256-LEFT.PL_3B/3B/3D/4B/7B
- new net MEM_D8: U1PE.PE11, U2MACHXO2-CSBGA132-640-LEFT.PL_/3C/4A/5A/8A
- new net MEM_D9: U1PE.PE12, U2MACHXO2-CSBGA132-640-LEFT.PL_/3D/4B/5B/8B
- new net MEM_NADV: U1PB.PB7
- new net MEM_NBL0: U1PE.PE0
- new net MEM_NBL1: U1PE.PE1
- new net MEM_NOE: U1PD.PD4
- new net MEM_NWAIT: U1PD.PD6
- new net MEM_NWE: U1PD.PD5
- new net MEM_SDCKE0: U1PC.PC3-ADC_IN13
- new net MEM_SDCLK: U1PG.PG8
- new net MEM_SDNCAS: U1PG.PG15
- new net MEM_SDNE0: U1PC.PC2-ADC_IN12
- new net MEM_SDNRAS: U1PF.PF11
- new net MEM_SDWNE: U1PC.PC0-ADC_IN10
- new net PROGRAMN: J3.32, U1PA.PA12, U1PC.PC8
- net +3V3: now also U1PWR.VBAT, U1PWR.VDD; no longer U3PWR.VBAT, U3PWR.VDD
- net BOOT0: now also U1CTL.BOOT0; no longer U3CTL.BOOT0
- net ETH_NRST: now also U4.NRST; no longer U1.NRST
- net ETH_RXER: now also U4.RXER; no longer U1.RXER
- net ETH_TXD0: now also U1PG.PG13, U4.TXD0; no longer U1.TXD0, U3PB.PB12
- net ETH_TXD1: now also U1PG.PG14, U4.TXD1; no longer U1.TXD1, U3PB.PB13
- net GNDI: now also U1PWR.VSS, U4.GND, X2.KL1; no longer SV6.5, U1.GND, U3PWR.VSS
- net N$10: now also U4.TX+; no longer SV6.4, U1.TX+
- net N$11: now also U4.TX-; no longer SV6.3, U1.TX-
- net N$2: now also U1PC.PC14-OSC32_IN; no longer U3PC.PC14-OSC32_IN
- net N$3: now also U1PC.PC15-OSC32_OUT; no longer U3PC.PC15-OSC32_OUT
- net N$4: now also U1PWR.VCAP1; no longer U3CTL.VCAP1
- net N$5: now also U1PWR.VCAP2; no longer U3CTL.VCAP2
- net N$7: now also U4.RX-; no longer SV6.1, U1.RX-
- net N$8: now also U4.RX+; no longer SV6.2, U1.RX+
- net N100630: now also U1PWR.VDDA; no longer U3PWR.VDDA
- net N98218: now also U1PWR.VSSA; no longer U3PWR.VSSA
- net NRES: now also U1CTL.NRST; no longer U3CTL.NRST
- net PF0: now also U1CTL.PH0-OSC_IN; no longer J4.8, U3CTL.PH0-OSC_IN, U3PF.PF0
- net PF1: now also U1CTL.PH1-OSC_OUT; no longer U3CTL.PH1-OSC_OUT
- net RTC: now also U1PC.PC13; no longer U3PC.PC13
- net V-POE: now also X1.KL1; no longer SV6.6
