File: PoElli/PoElli-at.brd (EAGLE design)
At the start: 100 x 80 mm, 129 parts, among them J1 DF12-ELLI-HEADER-TOP, J3 M022.54MM_SCREWTERM, J4 M022.54MM_SCREWTERM, Q1 SI1307DL, Q2 FDV301N, Q3 FDMC2674, T1 Coilcraft 230NL, T2 FLYBACK750311689, U1 ENC624J600-I/PT, U2 NCP1117, U3 FST3257, U4 LT3748, U5 TPS2378, X1 POE-TP-RJ45-MOLEX, Y1 25MHz

Commit message: Arrange PoElli testpoints
Parts:
- added D5: 5.1V TBD, SparkFun-DiscreteSemi:SMB-DIODE
- TP1: value TEST_POINT-BARE -> TEST_POINT-5000; device ELL-i-Passives:TP_BARE -> ELL-i-Passives:TP_5021
- TP10: value TEST_POINT-5000 -> TEST_POINT-BARE; device ELL-i-Passives:TP_5021 -> ELL-i-Passives:TP_BARE
- moved TP1 30.5 mm to (66.0, 53.3)
- moved TP10 30.5 mm to (44.5, 31.8)
Connections:
- removed net N$35: R37.2, SW1.3, SW1.4, U1.49
- removed net N$65: TP5.P$1
- removed net N$67: TP6.P$1
- removed net N$68: TP7.P$1
- removed net N$69: TP8.P$1
- removed net N$70: TP9.P$1
- removed net N$71: TP10.P$1
- new net ETH_SS: R37.2, SW1.3, SW1.4, TP2.P$1, U1.49
- net +3V3: now also TP7.P$1; no longer TP2.P$1
- net 5V: now also D5.C, TP8.P$1; no longer TP3.P$1
- net ETH_INT: now also TP6.P$1
- net ETH_MISO: now also TP5.P$1
- net ETH_MOSI: now also TP4.P$1
- net ETH_MUX: now also TP1.P$1
- net ETH_SCK: now also TP3.P$1
- net GNDA: now also D5.A, TP9.P$1; no longer TP4.P$1
- net SGND: now also TP10.P$1; no longer TP1.P$1
