File: PoElli/PoElli-at.sch (EAGLE design)
At the start: 121 parts, among them J1 DF12-ELLI-HEADER-TOP, Q1 SI1307DL, Q2 FDV301N, Q3 FDMC2674, T1 Coilcraft 230NL, T2 FLYBACK750311689, U1 ENC624J600-I/PT, U2 NCP1117, U3 FST3257, U4 LT3748, U5 TPS2378, X1 POE-TP-RJ45-MOLEX, Y1 25MHz

Commit message: Cleanups to PoElli schematics
Parts:
- FB2, FB3: value (none) -> 2A
Connections:
- net GND renamed RTN
- net N$15 renamed VSS
- net N$16 renamed VDD
Other:
- moved on the sheet: C10, C16, C17, C18, C19, C20, C21, C22, C23, C24, C25, C26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

Commit message: Further cleanups and add components to PoElli schematics
Parts:
- removed JP1: M022.54MM_SCREWTERM, SparkFun-Connectors:M022.54MM_SCREWTERM
- added C28: 33nF, ELL-i-Passives:C0805
- added C33: 150pF NP, ELL-i-Passives:C0805
- added D11: BAS70J, ELL-i-DIscreteSemi:BAS70J
- added D13: TBD 18V, SparkFun-DiscreteSemi:DIODE-ZENERSMB
- added J3, J4: M022.54MM_SCREWTERM, SparkFun-Connectors:M022.54MM_SCREWTERM
- added R25: 100K, ELL-i-Passives:R0603
- added R27: 220R, ELL-i-Passives:R1206
- added R38: 0R, ELL-i-Passives:R0603
- C38: value 470p -> 6n8; device ELL-i-Passives:C0805 -> ELL-i-Passives:C0402
- C39: value 6n8 -> 470p; device ELL-i-Passives:C0402 -> ELL-i-Passives:C0805
- D6: device TPS2378:BAS70J -> ELL-i-DIscreteSemi:BAS70J
Connections:
- net N$34 renamed UNREG_5V+
- removed net N$58: C16.-, C17.2, C18.2, C23.-, T2.SEC-, TP4.P$1, U2.GND
- new net GND: C28.1, R27.2
- new net N$10: J3.2
- new net N$15: C33.2, R27.1
- new net N$9: D11.C, D13.C, R25.2, R38.2, U5.CDB
- net GNDA: now also C16.-, C17.2, C18.2, C23.-, C28.2, T2.SEC-, TP4.P$1, U2.GND
- net N$17: now also D11.A
- net N$20: now also R38.1; no longer U5.CDB
- net N$22: now also C39.1; no longer C38.1
- net N$23: now also C38.1; no longer C39.1
- net N$28: now also C33.1
- net N$53: now also J4.2; no longer JP1.2
- net N$55: now also J4.1; no longer JP1.1
- net RTN: now also D13.A
- net VDD: now also J3.1, R25.1
Other:
- note added: "Add N-FET!"
- note added: "R38 solder bridge is a potential alternative to R25, D11 and D13. To be tested."
- note removed: "Add ground"
- moved on the sheet: C16, C17, C18, C21, C22, C23, C29, C3, C30, C32, C34, C35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

Commit message: Small cleanups to PoElli
Parts:
- R38: value 0R -> 0R NP
Other:
- note added: "1500V"
- moved on the sheet: C25, C26, C28, R19, R20
Changed lines of the file:
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@@
 <part name="SUPPLY5" library="SparkFun-Aesthetics" deviceset="5V" device=""/>
 <part name="U$1" library="SparkFun-Aesthetics" deviceset="FRAME-A4L" device=""/>
-<part name="R38" library="ELL-i-Passives" deviceset="R" device="0603" value="0R"/>
+<part name="R38" library="ELL-i-Passives" deviceset="R" device="0603" value="0R NP"/>
 <part name="R25" library="ELL-i-Passives" deviceset="R" device="0603" value="100K"/>
 <part name="D11" library="ELL-i-DIscreteSemi" deviceset="BAS70" device="J"/>
@@
 To be tested.</text>
 <text x="0" y="-15.24" size="1.778" layer="91">Add N-FET!</text>
+<text x="53.34" y="109.22" size="1.778" layer="97">1500V</text>
 </plain>
 <instances>
@@
 <instance part="GND16" gate="1" x="256.54" y="210.82"/>
 <instance part="R21" gate="G$1" x="-167.64" y="175.26" rot="R90"/>
-<instance part="R20" gate="G$1" x="-149.86" y="175.26" rot="R90"/>
-<instance part="R19" gate="G$1" x="-134.62" y="175.26" rot="R90"/>
+<instance part="R20" gate="G$1" x="-147.32" y="175.26" rot="R90"/>
+<instance part="R19" gate="G$1" x="-137.16" y="175.26" rot="R90"/>
 <instance part="R18" gate="G$1" x="-116.84" y="175.26" rot="R90"/>
 <instance part="C27" gate="G$1" x="-167.64" y="190.5"/>
-<instance part="C26" gate="G$1" x="-149.86" y="190.5"/>
-<instance part="C25" gate="G$1" x="-134.62" y="190.5"/>
+<instance part="C26" gate="G$1" x="-147.32" y="190.5" rot="MR0"/>
+<instance part="C25" gate="G$1" x="-137.16" y="190.5"/>
 <instance part="C24" gate="G$1" x="-116.84" y="190.5"/>
 <instance part="C31" gate="G$1" x="-142.24" y="157.48"/>
@@
 <instance part="R27" gate="G$1" x="55.88" y="45.72" rot="R270"/>
 <instance part="GND29" gate="1" x="55.88" y="33.02"/>
-<instance part="C28" gate="G$1" x="55.88" y="114.3" rot="R90"/>
+<instance part="C28" gate="G$1" x="54.356" y="114.3" rot="R90"/>
 <instance part="GND30" gate="1" x="71.12" y="109.22"/>
 <instance part="GND31" gate="1" x="43.18" y="109.22"/>
@@
 <wire x1="-162.56" y1="259.08" x2="-147.32" y2="259.08" width="0.1524" layer="91"/>
 <junction x="-147.32" y="259.08"/>
-<wire x1="-147.32" y1="259.08" x2="-147.32" y2="200.66" width="0.1524" layer="91"/>
-<wire x1="-147.32" y1="200.66" x2="-149.86" y2="200.66" width="0.1524" layer="91"/>
-<label x="-152.4" y="200.66" size="1.778" layer="95" rot="R180" xref="yes"/>
-<wire x1="-149.86" y1="200.66" x2="-152.4" y2="200.66" width="0.1524" layer="91"/>
-<wire x1="-149.86" y1="193.04" x2="-149.86" y2="200.66" width="0.1524" layer="91"/>
-<junction x="-149.86" y="200.66"/>
+<wire x1="-147.32" y1="259.08" x2="-147.32" y2="205.74" width="0.1524" layer="91"/>
+<label x="-162.56" y="200.66" size="1.778" layer="95" xref="yes"/>
+<wire x1="-147.32" y1="193.04" x2="-147.32" y2="205.74" width="0.1524" layer="91"/>
+<wire x1="-162.56" y1="200.66" x2="-165.1" y2="200.66" width="0.1524" layer="91"/>
+<wire x1="-165.1" y1="200.66" x2="-165.1" y2="205.74" width="0.1524" layer="91"/>
+<wire x1="-165.1" y1="205.74" x2="-147.32" y2="205.74" width="0.1524" layer="91"/>
+<junction x="-147.32" y="205.74"/>
 </segment>
 </net>
@@
 </segment>
 <segment>
-<wire x1="-134.62" y1="213.36" x2="-134.62" y2="208.28" width="0.1524" layer="91"/>
-<wire x1="-134.62" y1="208.28" x2="-132.08" y2="208.28" width="0.1524" layer="91"/>
+<wire x1="-134.62" y1="215.9" x2="-134.62" y2="210.82" width="0.1524" layer="91"/>
+<wire x1="-134.62" y1="210.82" x2="-132.08" y2="210.82" width="0.1524" layer="91"/>
 <pinref part="T1" gate="G$1" pin="TXCT"/>
 <wire x1="-132.08" y1="238.76" x2="-134.62" y2="238.76" width="0.1524" layer="91"/>
-<wire x1="-134.62" y1="238.76" x2="-134.62" y2="213.36" width="0.1524" layer="91"/>
-<junction x="-134.62" y="213.36"/>
-<wire x1="-116.84" y1="213.36" x2="-134.62" y2="213.36" width="0.1524" layer="91"/>
+<wire x1="-134.62" y1="238.76" x2="-134.62" y2="215.9" width="0.1524" layer="91"/>
+<junction x="-134.62" y="215.9"/>
+<wire x1="-116.84" y1="215.9" x2="-134.62" y2="215.9" width="0.1524" layer="91"/>
 <pinref part="C24" gate="G$1" pin="1"/>
-<wire x1="-116.84" y1="193.04" x2="-116.84" y2="213.36" width="0.1524" layer="91"/>
-<label x="-132.08" y="208.28" size="1.778" layer="95" xref="yes"/>
+<wire x1="-116.84" y1="193.04" x2="-116.84" y2="215.9" width="0.1524" layer="91"/>
+<label x="-132.08" y="210.82" size="1.778" layer="95" xref="yes"/>
 </segment>
 </net>
@@
 </segment>
 <segment>
-<wire x1="-137.16" y1="200.66" x2="-134.62" y2="200.66" width="0.1524" layer="91"/>
 <pinref part="T1" gate="G$1" pin="RXCT"/>
-<wire x1="-134.62" y1="200.66" x2="-132.08" y2="200.66" width="0.1524" layer="91"/>
+<wire x1="-137.16" y1="200.66" x2="-132.08" y2="200.66" width="0.1524" layer="91"/>
 <wire x1="-132.08" y1="259.08" x2="-137.16" y2="259.08" width="0.1524" layer="91"/>
 <wire x1="-137.16" y1="259.08" x2="-137.16" y2="200.66" width="0.1524" layer="91"/>
 <pinref part="C25" gate="G$1" pin="1"/>
 <label x="-132.08" y="200.66" size="1.778" layer="95" xref="yes"/>
-<wire x1="-134.62" y1="193.04" x2="-134.62" y2="200.66" width="0.1524" layer="91"/>
-<junction x="-134.62" y="200.66"/>
+<wire x1="-137.16" y1="193.04" x2="-137.16" y2="200.66" width="0.1524" layer="91"/>
+<junction x="-137.16" y="200.66"/>
 </segment>
 </net>
@@
 <junction x="-149.86" y="251.46"/>
 <pinref part="C27" gate="G$1" pin="1"/>
-<wire x1="-167.64" y1="193.04" x2="-167.64" y2="213.36" width="0.1524" layer="91"/>
-<wire x1="-167.64" y1="213.36" x2="-149.86" y2="213.36" width="0.1524" layer="91"/>
-<wire x1="-149.86" y1="213.36" x2="-149.86" y2="251.46" width="0.1524" layer="91"/>
-<label x="-152.4" y="208.28" size="1.778" layer="95" rot="R180" xref="yes"/>
-<wire x1="-149.86" y1="213.36" x2="-149.86" y2="208.28" width="0.1524" layer="91"/>
-<junction x="-149.86" y="213.36"/>
-<wire x1="-149.86" y1="208.28" x2="-152.4" y2="208.28" width="0.1524" layer="91"/>
+<wire x1="-167.64" y1="193.04" x2="-167.64" y2="210.82" width="0.1524" layer="91"/>
+<wire x1="-167.64" y1="210.82" x2="-167.64" y2="215.9" width="0.1524" layer="91"/>
+<wire x1="-167.64" y1="215.9" x2="-149.86" y2="215.9" width="0.1524" layer="91"/>
+<wire x1="-149.86" y1="215.9" x2="-149.86" y2="251.46" width="0.1524" layer="91"/>
+<label x="-162.56" y="210.82" size="1.778" layer="95" xref="yes"/>
+<wire x1="-162.56" y1="210.82" x2="-167.64" y2="210.82" width="0.1524" layer="91"/>
+<junction x="-167.64" y="210.82"/>
 </segment>
 </net>
@@
 <pinref part="C28" gate="G$1" pin="2"/>
 <pinref part="GND30" gate="1" pin="GNDA"/>
-<wire x1="60.96" y1="114.3" x2="71.12" y2="114.3" width="0.1524" layer="91"/>
+<wire x1="59.436" y1="114.3" x2="71.12" y2="114.3" width="0.1524" layer="91"/>
 <wire x1="71.12" y1="114.3" x2="71.12" y2="111.76" width="0.1524" layer="91"/>
 </segment>
@@
 <pinref part="R19" gate="G$1" pin="2"/>
 <pinref part="C25" gate="G$1" pin="2"/>
-<wire x1="-134.62" y1="180.34" x2="-134.62" y2="185.42" width="0.1524" layer="91"/>
+<wire x1="-137.16" y1="180.34" x2="-137.16" y2="185.42" width="0.1524" layer="91"/>
 </segment>
 </net>
@@
 <pinref part="C26" gate="G$1" pin="2"/>
 <pinref part="R20" gate="G$1" pin="2"/>
-<wire x1="-149.86" y1="185.42" x2="-149.86" y2="180.34" width="0.1524" layer="91"/>
+<wire x1="-147.32" y1="185.42" x2="-147.32" y2="180.34" width="0.1524" layer="91"/>
 </segment>
 </net>
@@
 <pinref part="C31" gate="G$1" pin="1"/>
 <pinref part="R19" gate="G$1" pin="1"/>
-<wire x1="-134.62" y1="170.18" x2="-134.62" y2="167.64" width="0.1524" layer="91"/>
+<wire x1="-137.16" y1="170.18" x2="-137.16" y2="167.64" width="0.1524" layer="91"/>
 <pinref part="R20" gate="G$1" pin="1"/>
 <pinref part="R21" gate="G$1" pin="1"/>
 <wire x1="-167.64" y1="170.18" x2="-167.64" y2="167.64" width="0.1524" layer="91"/>
-<wire x1="-167.64" y1="167.64" x2="-149.86" y2="167.64" width="0.1524" layer="91"/>
-<junction x="-149.86" y="167.64"/>
-<wire x1="-149.86" y1="167.64" x2="-142.24" y2="167.64" width="0.1524" layer="91"/>
-<wire x1="-142.24" y1="167.64" x2="-134.62" y2="167.64" width="0.1524" layer="91"/>
-<wire x1="-149.86" y1="170.18" x2="-149.86" y2="167.64" width="0.1524" layer="91"/>
+<wire x1="-167.64" y1="167.64" x2="-147.32" y2="167.64" width="0.1524" layer="91"/>
+<junction x="-147.32" y="167.64"/>
+<wire x1="-147.32" y1="167.64" x2="-142.24" y2="167.64" width="0.1524" layer="91"/>
+<wire x1="-142.24" y1="167.64" x2="-137.16" y2="167.64" width="0.1524" layer="91"/>
+<wire x1="-147.32" y1="170.18" x2="-147.32" y2="167.64" width="0.1524" layer="91"/>
 <pinref part="R18" gate="G$1" pin="1"/>
 <wire x1="-116.84" y1="167.64" x2="-116.84" y2="170.18" width="0.1524" layer="91"/>
-<wire x1="-134.62" y1="167.64" x2="-116.84" y2="167.64" width="0.1524" layer="91"/>
-<junction x="-134.62" y="167.64"/>
+<wire x1="-137.16" y1="167.64" x2="-116.84" y2="167.64" width="0.1524" layer="91"/>
+<junction x="-137.16" y="167.64"/>
 <wire x1="-142.24" y1="160.02" x2="-142.24" y2="167.64" width="0.1524" layer="91"/>
 <junction x="-142.24" y="167.64"/>
@@
 <pinref part="C28" gate="G$1" pin="1"/>
 <pinref part="GND31" gate="1" pin="GND"/>
-<wire x1="53.34" y1="114.3" x2="43.18" y2="114.3" width="0.1524" layer="91"/>
+<wire x1="51.816" y1="114.3" x2="43.18" y2="114.3" width="0.1524" layer="91"/>
 <wire x1="43.18" y1="114.3" x2="43.18" y2="111.76" width="0.1524" layer="91"/>
 </segment>

Commit message: Arrange PoElli testpoints
Parts:
- added D5: 5.1V TBD, SparkFun-DiscreteSemi:DIODE-ZENERSMB
- TP1: value TEST_POINT-BARE -> TEST_POINT-5000; device ELL-i-Passives:TEST_POINT-BARE -> ELL-i-Passives:TEST_POINT-5000
- TP10: value TEST_POINT-5000 -> TEST_POINT-BARE; device ELL-i-Passives:TEST_POINT-5000 -> ELL-i-Passives:TEST_POINT-BARE
Connections:
- removed net N$35: R37.2, SW1.3, SW1.4, U1.~CS/CS
- removed net N$65: TP5.P$1
- removed net N$67: TP6.P$1
- removed net N$68: TP7.P$1
- removed net N$69: TP8.P$1
- removed net N$70: TP9.P$1
- removed net N$71: TP10.P$1
- new net ETH_SS: R37.2, SW1.3, SW1.4, TP2.P$1, U1.~CS/CS
- net +3V3: now also TP7.P$1; no longer TP2.P$1
- net 5V: now also D5.C, TP8.P$1; no longer TP3.P$1
- net ETH_INT: now also TP6.P$1
- net ETH_MISO: now also TP5.P$1
- net ETH_MOSI: now also TP4.P$1
- net ETH_MUX: now also TP1.P$1
- net ETH_SCK: now also TP3.P$1
- net GNDA: now also D5.A, TP9.P$1; no longer TP4.P$1
- net SGND: now also TP10.P$1; no longer TP1.P$1
Other:
- note removed: "Add 5V1 zen"
- moved on the sheet: C16, C17, C18, C21, C22, C23, C28, C3, C33, D3, D4, D6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

Commit message: Change to ENC424J600 & cleanups in PoElli
Parts:
- removed U1: ENC624J600-I/PT, ELL-i-DigitalIC:ENC624J600-I/PT
- added U6: ENC424J600, ELL-i-DigitalIC:ENC424J600
Connections:
- net ENC-3V3: now also U6.VDD, U6.VDDOSC, U6.VDDPLL, U6.VDDRX, U6.VDDTX; no longer U1.VDD, U1.VDDOSC, U1.VDDPLL, U1.VDDRX, U1.VDDTX, U1.VDD_2, U1.VDD_3
- net ETH_INT: now also U6.!INT!/SPISEL; no longer U1.~INT/SPISEL
- net ETH_MISO: now also U6.SO/WR/EN; no longer U1.SO/WR/WRL/EN/BOSEL
- net ETH_MOSI: now also U6.SI/RD/!RW; no longer U1.SI/RD/R~W
- net ETH_SCK: now also U6.SCK/AL; no longer U1.SCK/AL/PSPCFG4
- net ETH_SS: now also U6.!CS!/CS; no longer U1.~CS/CS
- net GNDA: now also U6.AD0, U6.AD1, U6.AD10, U6.AD11, U6.AD12, U6.AD13, U6.AD14, U6.AD2, U6.AD3, U6.AD4, U6.AD5, U6.AD6, U6.AD7, U6.AD8, U6.AD9, U6.PSPCFG0, U6.VSS1, U6.VSS2, U6.VSSOSC, U6.VSSPLL, U6.VSSRX, U6.VSSTX1, U6.VSSTX2; no longer U1.A0, U1.A1, U1.A10, U1.A11, U1.A12, U1.A13, U1.A14/PSPCFG1, U1.A2, U1.A3, U1.A4, U1.A5, U1.A6, U1.A7, U1.A8, U1.A9, U1.AD0, U1.AD1, U1.AD10, U1.AD11, U1.AD12, U1.AD13, U1.AD14, U1.AD15, U1.AD2, U1.AD3, U1.AD4, U1.AD5, U1.AD6, U1.AD7, U1.AD8, U1.AD9, U1.PSPCFG2, U1.PSPCFG3, U1.VSS, U1.VSSOSC, U1.VSSPLL, U1.VSSRX, U1.VSSTX, U1.VSSTX1, U1.VSS_2, U1.WRH/B1SEL
- net N$37: now also U6.OSC2; no longer U1.OSC2
- net N$39: now also U6.TPIN-; no longer U1.TPIN-
- net N$41: now also U6.LEDB; no longer U1.LEDB
- net N$42: now also U6.LEDA; no longer U1.LEDA
- net N$45: now also U6.RBIAS; no longer U1.RBIAS
- net N$46: now also U6.VCAP; no longer U1.VCAP
- net N$47: now also U6.OSC1; no longer U1.OSC1
- net N$59: now also U6.TPIN+; no longer U1.TPIN+
- net TPOUT+: now also R13.1, U6.TPOUT+; no longer R12.1, U1.TPOUT-
- net TPOUT-: now also R12.1, U6.TPOUT-; no longer R13.1, U1.TPOUT+
Other:
- moved on the sheet: C1, C11, C12, C13, C14, C15, C2, C4, C5, C6, C7, C8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

Commit message: Initial layout for PoElli
Parts:
- SV1: value RASPBERRYPI-GPIOPTH -> RASPBERRY-SHIELD; device SparkFun-Boards:RASPBERRYPI-GPIOPTH -> ELL-i-Boards:RASPBERRY-SHIELD
- X1: value POE-TP-RJ45-MOLEX -> RJ45
- renumbered XXR35XX to R39
Other:
- moved on the sheet: SW1

Commit message: Review changes to PoElli-at
Parts:
- removed D1: (no value), SparkFun-LED:LED-YELLOW0603
- removed D2: GREEN, SparkFun-LED:LED-GREEN0603
- removed R11: 0R, ELL-i-Passives:R0805
- removed TP10: TEST_POINT-BARE, ELL-i-Passives:TEST_POINT-BARE
- added C36: 47p, ELL-i-Passives:C0402
- added C43, C44, C45, C46, C47: 22uF, ELL-i-Passives:C0805
- added C48: 1nF, ELL-i-Passives:CC1206
- added D19: B2100, ELL-i-DIscreteSemi:DIODE-SCHOTTKYB2100
- added Q4: IRFL4310, ELL-i-DIscreteSemi:IRFL4310
- added SJ1: CLOSED, SparkFun-Passives:SOLDERJUMPERNC
- added SJ2, SJ3: OPEN, SparkFun-Passives:SOLDERJUMPERNO
- C1, C2, C37: device ELL-i-Passives:C0603 -> ELL-i-Passives:C0402
- C10, C11, C12, C14, C15, C17, C18, C19, C20, C3, C39, C4, C5, C6, C7, C8, C9: device ELL-i-Passives:C0805 -> ELL-i-Passives:C0402
- C16: value 47u -> 47uF; device ELL-i-Passives:CPOL6032 -> ELL-i-Passives:CPOL1206
- C22, C24, C25, C26, C27, C34, C40, C42: device ELL-i-Passives:C0805 -> ELL-i-Passives:C0603
- C23: value (none) -> 220uF; device ELL-i-Passives:CPOLC -> ELL-i-Passives:CPOLE
- C28: value 33nF -> 1nF; device ELL-i-Passives:C0805 -> ELL-i-Passives:CC1206
- C31: device ELL-i-Passives:C0805 -> ELL-i-Passives:C1210
- C32: device ELL-i-Passives:C0805 -> ELL-i-Passives:CPOL1206
- D12: device ell-i:SMAJ58A -> ELL-i-DIscreteSemi:SMAJ58A
- D13: value TBD 18V -> 18V; device SparkFun-DiscreteSemi:DIODE-ZENERSMB -> ELL-i-DIscreteSemi:DIODE-ZENER-SOD-123
- D5: value 5.1V TBD -> 5.6V TBD; device SparkFun-DiscreteSemi:DIODE-ZENERSMB -> ELL-i-DIscreteSemi:DIODE-ZENER-SOD-123
- FB1: device ELL-i-Passives:FB -> ELL-i-Passives:FB0402
- FB2, FB3, FB4, FB5: device ELL-i-Passives:FB -> ELL-i-Passives:FB1206
- J3, J4: value M022.54MM_SCREWTERM -> M022.54MM
- R1, R12, R13, R14, R17, R2, R7, R8, R9: device ELL-i-Passives:R0805 -> ELL-i-Passives:R0402
- R10: value 0R -> 100; device ELL-i-Passives:R0805 -> ELL-i-Passives:R0603
- R15, R18, R19, R20, R21, R35, R36, R5: device ELL-i-Passives:R0805 -> ELL-i-Passives:R0603
- R16: device ELL-i-Passives:R0805 -> ELL-i-Passives:R1206
- R22, R23, R24, R26, R30, R31, R33, R34: device ELL-i-Passives:R0402 -> ELL-i-Passives:R0603
- R27, R32: device ELL-i-Passives:R1206 -> ELL-i-Passives:R0805
- R29: device ELL-i-Passives:R0402 -> ELL-i-Passives:R0805
- R3, R4: value 180 -> 330
- R38: value 0R NP -> OPEN; device ELL-i-Passives:R0603 -> SparkFun-Passives:SOLDERJUMPERNO
- R6: device ELL-i-Passives:R0603 -> ELL-i-Passives:R0402
- U2: device ell-i:NCP1117 -> ELL-i-PowerIC:NCP1117
- X1: value RJ45 -> XMK-8788K5-BX1X; device ELL-i-Connectors:POE-TP-RJ45-MOLEX -> ELL-i-Connectors:POE-TP-SHIELDED-LEDS
- Y1: value 25MHz -> 25 MHz; device SparkFun-FreqCtrl:CRYSTAL5X3 -> SparkFun-FreqCtrl:CRYSTAL_WITH_GND
Connections:
- removed net GND: C28.1, R27.2
- new net N$21: D19.C, J3.1
- new net N$34: C21.2, R10.2
- new net N$35: J1.VCC(IO), SJ3.1
- net +3V3: now also SJ1.2, SJ3.2; no longer R10.2
- net +5V0: now also SJ2.2; no longer R11.2
- net 5V: now also C43.1, C44.1, C45.1, C46.1, C47.1
- net GNDA: now also C43.2, C44.2, C45.2, C46.2, C47.2, C48.2, X1LED1.C, X1LED2.C, Y1.GND@1, Y1.GND@2; no longer D1.C, D2.C
- net N$1: now also X1RJ45.TX-@2; no longer X1.TX-@2
- net N$10: now also Q4.D
- net N$2: now also X1RJ45.TX+@1; no longer X1.TX+@1
- net N$26: now also C36.1
- net N$3: now also X1RJ45.RX+@3; no longer X1.RX+@3
- net N$33: now also R10.1; no longer C21.2
- net N$36: now also X1LED2.A; no longer D1.A
- net N$37: now also Y1.C1; no longer Y1.1
- net N$38: now also X1LED1.A; no longer D2.A
- net N$4: now also X1RJ45.RX-@6; no longer X1.RX-@6
- net N$43: now also SJ1.1, SJ2.1; no longer R10.1, R11.1
- net N$47: now also Y1.C2; no longer Y1.2
- net N$9: now also Q4.G
- net POE_B+: now also X1RJ45.POE+@4, X1RJ45.POE+@5; no longer X1.POE+@4, X1.POE+@5
- net POE_B-: now also X1RJ45.POE-@7, X1RJ45.POE-@8; no longer X1.POE-@7, X1.POE-@8
- net RTN: now also C28.1, C32.-, C36.2, C48.1, Q4.S, R27.2, X1RJ45.GND@0, X1RJ45.GND@2; no longer C32.2
- net SGND: no longer TP10.P$1
- net VDD: now also C32.+, D19.A; no longer C32.1, J3.1
Other:
- note added: "10V H6.2mm"
- note added: "200V"
- note added: "Allow manual replacement of R29"
- note added: "C10 and C19 close to transformer pins"
- note added: "Enable manual replacement of R39 and R37"
- note added: "Leds to the RJ-45 connector?"
- note added: "TODO: - Review XMK RJ-45 connector - Review SOT-323 and SOT-23 layouts"
- note added: "XMK-8788K5-BX1X 1.5A Offset mounted connector Assembly normally (not upside down)"
- note removed: "1500V"
- note removed: "Add N-FET!"
- note removed: "VCC(IO) left open"
- note removed: "WRONG FOOTPRINT FOR Y1"
- moved on the sheet: C1, C10, C16, C17, C18, C19, C2, C21, C23, C28, C29, C30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
