File: PoElli/PoElli-at.sch (EAGLE design)
At the start: 138 parts, among them J1 DF12-ELLI-HEADER-TOP, J3 M022.54MM, J4 M022.54MM, Q1 SI1307DL, Q2 FDV301N, Q3 FDMC2674, Q4 IRFL4310, T1 Coilcraft 230NL, T2 FLYBACK750311689, U2 NCP1117, U3 FST3257, U4 LT3748, U5 TPS2378, U6 ENC424J600, X1 XMK-8788K5-BX1X, Y1 25 MHz

Commit message: Mechanical design
Parts:
- added JP1: XMK-8788K5-BX1X, ELL-i-Connectors:POE-TP-SHIELDED-LEDS
- added X2, X3, X4: M-BOLT-2, ELL-i-Connectors:M-BOLT-2
- X1: value XMK-8788K5-BX1X -> M-BOLT-2; device ELL-i-Connectors:POE-TP-SHIELDED-LEDS -> ELL-i-Connectors:M-BOLT-2
Connections:
- net 5V: now also X1.KL1
- net GNDA: now also JP1LED1.C, JP1LED2.C, X2.KL1; no longer X1LED1.C, X1LED2.C
- net N$1: now also JP1RJ45.TX-@2; no longer X1RJ45.TX-@2
- net N$2: now also JP1RJ45.TX+@1; no longer X1RJ45.TX+@1
- net N$3: now also JP1RJ45.RX+@3; no longer X1RJ45.RX+@3
- net N$36: now also JP1LED2.A; no longer X1LED2.A
- net N$38: now also JP1LED1.A; no longer X1LED1.A
- net N$4: now also JP1RJ45.RX-@6; no longer X1RJ45.RX-@6
- net POE_B+: now also JP1RJ45.POE+@4, JP1RJ45.POE+@5; no longer X1RJ45.POE+@4, X1RJ45.POE+@5
- net POE_B-: now also JP1RJ45.POE-@7, JP1RJ45.POE-@8; no longer X1RJ45.POE-@7, X1RJ45.POE-@8
- net RTN: now also JP1RJ45.GND@0, JP1RJ45.GND@2, X4.KL1; no longer X1RJ45.GND@0, X1RJ45.GND@2
- net VDD: now also X3.KL1
Changed lines of the file:
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@@
 <part name="R10" library="ELL-i-Passives" deviceset="R" device="0603" value="100"/>
 <part name="SJ3" library="SparkFun-Passives" deviceset="SOLDERJUMPER" device="NO" value="OPEN"/>
-<part name="X1" library="ELL-i-Connectors" deviceset="POE-TP-SHIELDED-LEDS" device="" value="XMK-8788K5-BX1X"/>
+<part name="JP1" library="ELL-i-Connectors" deviceset="POE-TP-SHIELDED-LEDS" device="" value="XMK-8788K5-BX1X"/>
+<part name="X1" library="ELL-i-Connectors" deviceset="M-BOLT" device="-2"/>
+<part name="X2" library="ELL-i-Connectors" deviceset="M-BOLT" device="-2"/>
+<part name="X3" library="ELL-i-Connectors" deviceset="M-BOLT" device="-2"/>
+<part name="X4" library="ELL-i-Connectors" deviceset="M-BOLT" device="-2"/>
+<part name="SUPPLY10" library="SparkFun-Aesthetics" deviceset="VDD" device=""/>
+<part name="GND5" library="supply1" deviceset="GNDA" device=""/>
+<part name="SUPPLY11" library="SparkFun-Aesthetics" deviceset="5V" device=""/>
 </parts>
 <sheets>
@@
 <instance part="R10" gate="G$1" x="7.62" y="101.6" rot="R180"/>
 <instance part="SJ3" gate="1" x="297.18" y="246.38" rot="R90"/>
-<instance part="X1" gate="RJ45" x="-170.18" y="251.46" rot="R180"/>
-<instance part="X1" gate="LED2" x="177.8" y="180.34" rot="R90"/>
-<instance part="X1" gate="LED1" x="187.96" y="180.34" rot="R90"/>
+<instance part="JP1" gate="RJ45" x="-170.18" y="251.46" rot="R180"/>
+<instance part="JP1" gate="LED2" x="177.8" y="180.34" rot="R90"/>
+<instance part="JP1" gate="LED1" x="187.96" y="180.34" rot="R90"/>
+<instance part="X1" gate="M" x="55.88" y="15.24"/>
+<instance part="X2" gate="M" x="55.88" y="7.62"/>
+<instance part="X3" gate="M" x="55.88" y="0"/>
+<instance part="X4" gate="M" x="57.658" y="-5.08" rot="MR0"/>
+<instance part="SUPPLY10" gate="VDD" x="71.12" y="5.08"/>
+<instance part="GND5" gate="1" x="63.5" y="2.54"/>
+<instance part="SUPPLY11" gate="G$1" x="63.5" y="17.78"/>
 </instances>
 <busses>
@@
 <pinref part="T1" gate="G$1" pin="TX-"/>
 <wire x1="-162.56" y1="246.38" x2="-132.08" y2="246.38" width="0.1524" layer="91"/>
-<pinref part="X1" gate="RJ45" pin="TX-@2"/>
+<pinref part="JP1" gate="RJ45" pin="TX-@2"/>
 </segment>
 </net>
@@
 <pinref part="T1" gate="G$1" pin="TX+"/>
 <wire x1="-142.24" y1="231.14" x2="-132.08" y2="231.14" width="0.1524" layer="91"/>
-<pinref part="X1" gate="RJ45" pin="TX+@1"/>
+<pinref part="JP1" gate="RJ45" pin="TX+@1"/>
 </segment>
 </net>
@@
 <pinref part="T1" gate="G$1" pin="RX+"/>
 <wire x1="-142.24" y1="251.46" x2="-132.08" y2="251.46" width="0.1524" layer="91"/>
-<pinref part="X1" gate="RJ45" pin="RX+@3"/>
+<pinref part="JP1" gate="RJ45" pin="RX+@3"/>
 </segment>
 </net>
@@
 <pinref part="T1" gate="G$1" pin="RX-"/>
 <wire x1="-142.24" y1="266.7" x2="-132.08" y2="266.7" width="0.1524" layer="91"/>
-<pinref part="X1" gate="RJ45" pin="RX-@6"/>
+<pinref part="JP1" gate="RJ45" pin="RX-@6"/>
 </segment>
 </net>
@@
 <wire x1="-165.1" y1="205.74" x2="-147.32" y2="205.74" width="0.1524" layer="91"/>
 <junction x="-147.32" y="205.74"/>
-<pinref part="X1" gate="RJ45" pin="POE-@7"/>
-<pinref part="X1" gate="RJ45" pin="POE-@8"/>
+<pinref part="JP1" gate="RJ45" pin="POE-@7"/>
+<pinref part="JP1" gate="RJ45" pin="POE-@8"/>
 </segment>
 </net>
@@
 <junction x="5.08" y="-5.08"/>
 <pinref part="Q4" gate="G$1" pin="S"/>
+<pinref part="X4" gate="M" pin="KL1"/>
+<wire x1="52.578" y1="-5.08" x2="33.02" y2="-5.08" width="0.1524" layer="91"/>
+<junction x="33.02" y="-5.08"/>
 </segment>
 <segment>
@@
 <segment>
 <pinref part="SUPPLY9" gate="G$1" pin="RTN"/>
-<pinref part="X1" gate="RJ45" pin="GND@2"/>
+<pinref part="JP1" gate="RJ45" pin="GND@2"/>
 <wire x1="-167.64" y1="231.14" x2="-167.64" y2="236.22" width="0.1524" layer="91"/>
 <wire x1="-167.64" y1="236.22" x2="-167.64" y2="238.76" width="0.1524" layer="91"/>
@@
 <wire x1="-185.42" y1="236.22" x2="-185.42" y2="271.78" width="0.1524" layer="91"/>
 <wire x1="-185.42" y1="271.78" x2="-167.64" y2="271.78" width="0.1524" layer="91"/>
-<pinref part="X1" gate="RJ45" pin="GND@0"/>
+<pinref part="JP1" gate="RJ45" pin="GND@0"/>
 <wire x1="-167.64" y1="271.78" x2="-167.64" y2="266.7" width="0.1524" layer="91"/>
 </segment>
@@
 <wire x1="195.58" y1="-15.24" x2="195.58" y2="0" width="0.1524" layer="91"/>
 </segment>
+<segment>
+<pinref part="X1" gate="M" pin="KL1"/>
+<wire x1="60.96" y1="15.24" x2="63.5" y2="15.24" width="0.1524" layer="91"/>
+<pinref part="SUPPLY11" gate="G$1" pin="5V"/>
+<wire x1="63.5" y1="15.24" x2="63.5" y2="17.78" width="0.1524" layer="91"/>
+</segment>
 </net>
 <net name="POE_A+" class="0">
@@
 <wire x1="-165.1" y1="210.82" x2="-167.64" y2="210.82" width="0.1524" layer="91"/>
 <junction x="-167.64" y="210.82"/>
-<pinref part="X1" gate="RJ45" pin="POE+@4"/>
-<pinref part="X1" gate="RJ45" pin="POE+@5"/>
+<pinref part="JP1" gate="RJ45" pin="POE+@4"/>
+<pinref part="JP1" gate="RJ45" pin="POE+@5"/>
 </segment>
 </net>
@@
 <wire x1="177.8" y1="177.8" x2="177.8" y2="175.26" width="0.1524" layer="91"/>
 <pinref part="GND8" gate="1" pin="GNDA"/>
-<pinref part="X1" gate="LED2" pin="C"/>
+<pinref part="JP1" gate="LED2" pin="C"/>
 </segment>
 <segment>
 <wire x1="187.96" y1="177.8" x2="187.96" y2="175.26" width="0.1524" layer="91"/>
 <pinref part="GND9" gate="1" pin="GNDA"/>
-<pinref part="X1" gate="LED1" pin="C"/>
+<pinref part="JP1" gate="LED1" pin="C"/>
 </segment>
 <segment>
@@
 <wire x1="210.82" y1="-22.86" x2="210.82" y2="-25.4" width="0.1524" layer="91"/>
 </segment>
+<segment>
+<pinref part="GND5" gate="1" pin="GNDA"/>
+<wire x1="63.5" y1="5.08" x2="63.5" y2="7.62" width="0.1524" layer="91"/>
+<pinref part="X2" gate="M" pin="KL1"/>
+<wire x1="63.5" y1="7.62" x2="60.96" y2="7.62" width="0.1524" layer="91"/>
+</segment>
 </net>
 <net name="N$36" class="0">
@@
 <pinref part="R4" gate="G$1" pin="2"/>
 <wire x1="177.8" y1="187.96" x2="177.8" y2="185.42" width="0.1524" layer="91"/>
-<pinref part="X1" gate="LED2" pin="A"/>
+<pinref part="JP1" gate="LED2" pin="A"/>
 </segment>
 </net>
@@
 <pinref part="R3" gate="G$1" pin="1"/>
 <wire x1="187.96" y1="187.96" x2="187.96" y2="185.42" width="0.1524" layer="91"/>
-<pinref part="X1" gate="LED1" pin="A"/>
+<pinref part="JP1" gate="LED1" pin="A"/>
 </segment>
 </net>
@@
 <wire x1="-10.16" y1="101.6" x2="-7.62" y2="101.6" width="0.1524" layer="91"/>
 <pinref part="T2" gate="G$1" pin="PRI-"/>
-<wire x1="-124.46" y1="2.54" x2="-124.46" y2="86.36" width="0.1524" layer="91"/>
+<wire x1="-124.46" y1="2.54" x2="-124.46" y2="83.82" width="0.1524" layer="91"/>
 <junction x="-124.46" y="86.36"/>
 <label x="-86.36" y="88.9" size="1.778" layer="95" rot="R180"/>
+<wire x1="-124.46" y1="83.82" x2="-124.46" y2="86.36" width="0.1524" layer="91"/>
 <wire x1="-15.24" y1="86.36" x2="-15.24" y2="78.74" width="0.1524" layer="91"/>
 <wire x1="-15.24" y1="78.74" x2="-15.24" y2="66.04" width="0.1524" layer="91"/>
@@
 <junction x="-58.42" y="86.36"/>
 <pinref part="SUPPLY6" gate="VDD" pin="VDD"/>
-<wire x1="-124.46" y1="91.44" x2="-124.46" y2="86.36" width="0.1524" layer="91"/>
+<wire x1="-124.46" y1="91.44" x2="-124.46" y2="88.9" width="0.1524" layer="91"/>
+<wire x1="-124.46" y1="88.9" x2="-124.46" y2="86.36" width="0.1524" layer="91"/>
 <wire x1="-10.16" y1="93.98" x2="-10.16" y2="86.36" width="0.1524" layer="91"/>
 <junction x="-10.16" y="86.36"/>
+<wire x1="-124.46" y1="88.9" x2="-124.46" y2="83.82" width="0.1524" layer="91"/>
 </segment>
 <segment>
@@
 <wire x1="35.56" y1="-20.32" x2="22.86" y2="-20.32" width="0.1524" layer="91"/>
 </segment>
-</net>
+<segment>
+<pinref part="X3" gate="M" pin="KL1"/>
+<wire x1="60.96" y1="0" x2="71.12" y2="0" width="0.1524" layer="91"/>
+<pinref part="SUPPLY10" gate="VDD" pin="VDD"/>
+<wire x1="71.12" y1="0" x2="71.12" y2="5.08" width="0.1524" layer="91"/>
+</segment>
+</net>
