File: PoElli/PoElli-Nucleo.sch (EAGLE design)
At the start: 120 parts, among them J3 M022.54MM, J4 M022.54MM, Q3 FDMC2674, Q4 IRFL4310, T1 Coilcraft 230NL, T2 FLYBACK750311689, U4 LT3748, U5 TPS2378, U6 ENC424J600, X1 RJ45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

Commit message: More work on Nucleo
Parts:
- removed D1: (no value), SparkFun-LED:LED-YELLOW0603
- removed D2: GREEN, SparkFun-LED:LED-GREEN0603
- removed TP8: TEST_POINT-5000, ELL-i-Passives:TEST_POINT-5000
- removed U$2: NUCLEO-SHIELD, ELL-i-Boards:NUCLEO-SHIELD
- removed X1: RJ45, ELL-i-Connectors:POE-TP-RJ45-MOLEX
- added J1: NUCLEO-SHIELD-NORMAL, ELL-i-Boards:NUCLEO-SHIELD-NORMAL
- added SW2: (no value), SparkFun-Electromechanical:SW_DIP-2-SMT-HALFSIZE
- added U$1: XMK-8788K5-BX1X, ELL-i-Connectors:POE-TP-SHIELDED-LEDS
Connections:
- removed net 5V: TP8.P$1
- net +3V3: now also J1CN7.3V3_12, J1CN7.3V3_16, R12.2, R13.2; no longer U$2ARDUINO.3.3V
- net ENC-3V3: no longer R12.2, R13.2
- net ETH_INT: now also SW2.3, SW2.4
- net ETH_MISO: now also J1CN10.PB14_28
- net ETH_MOSI: now also J1CN10.PB15_26
- net ETH_SCK: now also J1CN10.PB13_30
- net GNDA: now also J1CN7.GND_22, U$1LED1.C, U$1LED2.C; no longer D1.C, D2.C, U$2ARDUINO.GND@0, U$2ARDUINO.GND@1
- net N$1: now also U$1RJ45.TX-@2; no longer X1.TX-@2
- net N$11: now also J1CN7.1_PC10, SW1.2; no longer T1.TD+
- net N$12: now also J1CN7.3_PC12, SW1.1; no longer T1.TD-
- net N$13: now also J1CN7.PC11_2, SW2.1; no longer T1.RD+
- net N$14: now also J1CN7.PD2_4, SW2.2; no longer T1.RD-
- net N$2: now also U$1RJ45.TX+@1; no longer X1.TX+@1
- net N$3: now also U$1RJ45.RX+@3; no longer X1.RX+@3
- net N$36: now also U$1LED2.A; no longer D1.A
- net N$38: now also U$1LED1.A; no longer D2.A
- net N$4: now also U$1RJ45.RX-@6; no longer X1.RX-@6
- net POE_B+: now also U$1RJ45.POE+@4, U$1RJ45.POE+@5; no longer X1.POE+@4, X1.POE+@5
- net POE_B-: now also U$1RJ45.POE-@7, U$1RJ45.POE-@8; no longer X1.POE-@7, X1.POE-@8
- net RTN: now also U$1RJ45.GND@0, U$1RJ45.GND@2
- net TPIN+: now also T1.RD+
- net TPIN-: now also T1.RD-
- net TPOUT+: now also T1.TD+
- net TPOUT-: now also T1.TD-
- net VIN: now also J1CN7.VIN_24; no longer U$2ARDUINO.VIN
Other:
- note removed: "Enable manual replacement of R39 and R37"
- note removed: "TODO: - RJ-45 connector"
- moved on the sheet: C1, C11, C12, C13, C14, C15, C2, C22, C23, C4, C43, C44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

Commit message: Preliminary work on PoElli Nucleo layout
Parts:
- removed J1: NUCLEO-SHIELD-NORMAL, ELL-i-Boards:NUCLEO-SHIELD-NORMAL
- removed TP10: TEST_POINT-BARE, ELL-i-Passives:TEST_POINT-BARE
- added CN10: NUCLEO-CN10, ELL-i-Boards:NUCLEO-CN10
- added CN7: NUCLEO-CN7, ELL-i-Boards:NUCLEO-CN7
- added NUCLEO: NUCLEO-SHIELD-OUTLINE-EXTENDED, ELL-i-Boards:NUCLEO-SHIELD-OUTLINE-EXTENDED
Connections:
- removed net UNREG_5V+: C22.2, D4.A
- net +3V3: now also CN7.3V3_12, CN7.3V3_16; no longer J1CN7.3V3_12, J1CN7.3V3_16
- net ETH_MISO: now also CN10.27_PB4; no longer J1CN10.PB14_28
- net ETH_MOSI: now also CN10.25_PB10; no longer J1CN10.PB15_26
- net ETH_SCK: now also CN10.29_PB5; no longer J1CN10.PB13_30
- net GNDA: now also CN7.GND_22; no longer J1CN7.GND_22
- net N$11: now also CN7.1_PC10; no longer J1CN7.1_PC10
- net N$12: now also CN7.3_PC12; no longer J1CN7.3_PC12
- net N$13: now also CN7.PC11_2; no longer J1CN7.PC11_2
- net N$14: now also CN7.PD2_4; no longer J1CN7.PD2_4
- net SGND: no longer TP10.P$1
- net UNREG_6V+: now also C22.2, D4.A
- net VIN: now also CN7.VIN_24; no longer J1CN7.VIN_24

Commit message: Work on PoElli Nucleo
Parts:
- removed U$1: XMK-8788K5-BX1X, ELL-i-Connectors:POE-TP-SHIELDED-LEDS
- added D1: GREEN, SparkFun-LED:LED-GREEN0603
- added D2: YELLOW, SparkFun-LED:LED-YELLOW0603
- added X1: POE-TP-SHIELDED-RJ45-MOLEX-85502-5008, ELL-i-Connectors:POE-TP-SHIELDED-RJ45-MOLEX-85502-5008
Connections:
- net N$17 renamed U4_EN
- net N$20 renamed U4_SS
- net N$30 renamed INTVCC
- net N$9 renamed U5_CDB
- net GNDA: now also D1.C, D2.C; no longer U$1LED1.C, U$1LED2.C
- net N$1: now also X1.TX-@2; no longer U$1RJ45.TX-@2
- net N$2: now also X1.TX+@1; no longer U$1RJ45.TX+@1
- net N$3: now also X1.RX+@3; no longer U$1RJ45.RX+@3
- net N$36: now also D1.A; no longer U$1LED2.A
- net N$38: now also D2.A; no longer U$1LED1.A
- net N$4: now also X1.RX-@6; no longer U$1RJ45.RX-@6
- net POE_B+: now also X1.POE+@4, X1.POE+@5; no longer U$1RJ45.POE+@4, U$1RJ45.POE+@5
- net POE_B-: now also X1.POE-@7, X1.POE-@8; no longer U$1RJ45.POE-@7, U$1RJ45.POE-@8
- net RTN: now also X1.GND@0, X1.GND@2; no longer U$1RJ45.GND@0, U$1RJ45.GND@2
Changed lines of the file:
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@@
 <part name="+3V4" library="supply1" deviceset="+3V3" device=""/>
 <part name="SW2" library="SparkFun-Electromechanical" deviceset="SW_DIP-2" device="-SMT-HALFSIZE"/>
-<part name="U$1" library="ELL-i-Connectors" deviceset="POE-TP-SHIELDED-LEDS" device="" value="XMK-8788K5-BX1X"/>
 <part name="CN7" library="ELL-i-Boards" deviceset="NUCLEO-CN7" device=""/>
 <part name="CN10" library="ELL-i-Boards" deviceset="NUCLEO-CN10" device=""/>
 <part name="NUCLEO" library="ELL-i-Boards" deviceset="NUCLEO-SHIELD-OUTLINE" device="-EXTENDED"/>
+<part name="X1" library="ELL-i-Connectors" deviceset="POE-TP-SHIELDED" device="-RJ45-MOLEX-85502-5008"/>
+<part name="D1" library="SparkFun-LED" deviceset="LED-GREEN" device="0603" value="GREEN"/>
+<part name="D2" library="SparkFun-LED" deviceset="LED-YELLOW" device="0603" value="YELLOW"/>
 </parts>
 <sheets>
@@
 <instance part="+3V4" gate="G$1" x="114.3" y="208.28"/>
 <instance part="SW2" gate="G$1" x="281.94" y="304.8"/>
-<instance part="U$1" gate="RJ45" x="-165.1" y="251.46" rot="R180"/>
-<instance part="U$1" gate="LED2" x="185.42" y="177.8" rot="R90"/>
-<instance part="U$1" gate="LED1" x="195.58" y="177.8" rot="R90"/>
 <instance part="CN7" gate="CN7" x="322.58" y="271.78"/>
 <instance part="CN10" gate="CN10" x="322.58" y="210.82"/>
 <instance part="NUCLEO" gate="G$1" x="322.58" y="167.64"/>
+<instance part="X1" gate="G$1" x="-165.1" y="251.46" rot="R180"/>
+<instance part="D1" gate="G$1" x="185.42" y="180.34"/>
+<instance part="D2" gate="G$1" x="195.58" y="180.34"/>
 </instances>
 <busses>
@@
 <pinref part="T1" gate="G$1" pin="TX-"/>
 <wire x1="-157.48" y1="246.38" x2="-132.08" y2="246.38" width="0.1524" layer="91"/>
-<pinref part="U$1" gate="RJ45" pin="TX-@2"/>
+<pinref part="X1" gate="G$1" pin="TX-@2"/>
 </segment>
 </net>
@@
 <pinref part="T1" gate="G$1" pin="TX+"/>
 <wire x1="-142.24" y1="231.14" x2="-132.08" y2="231.14" width="0.1524" layer="91"/>
-<pinref part="U$1" gate="RJ45" pin="TX+@1"/>
+<pinref part="X1" gate="G$1" pin="TX+@1"/>
 </segment>
 </net>
@@
 <pinref part="T1" gate="G$1" pin="RX+"/>
 <wire x1="-142.24" y1="251.46" x2="-132.08" y2="251.46" width="0.1524" layer="91"/>
-<pinref part="U$1" gate="RJ45" pin="RX+@3"/>
+<pinref part="X1" gate="G$1" pin="RX+@3"/>
 </segment>
 </net>
@@
 <pinref part="T1" gate="G$1" pin="RX-"/>
 <wire x1="-142.24" y1="266.7" x2="-132.08" y2="266.7" width="0.1524" layer="91"/>
-<pinref part="U$1" gate="RJ45" pin="RX-@6"/>
+<pinref part="X1" gate="G$1" pin="RX-@6"/>
 </segment>
 </net>
@@
 <wire x1="-165.1" y1="205.74" x2="-147.32" y2="205.74" width="0.1524" layer="91"/>
 <junction x="-147.32" y="205.74"/>
-<pinref part="U$1" gate="RJ45" pin="POE-@7"/>
-<pinref part="U$1" gate="RJ45" pin="POE-@8"/>
+<pinref part="X1" gate="G$1" pin="POE-@7"/>
+<pinref part="X1" gate="G$1" pin="POE-@8"/>
 </segment>
 </net>
@@
 </segment>
 </net>
-<net name="N$17" class="0">
+<net name="U4_EN" class="0">
 <segment>
 <wire x1="-33.02" y1="71.12" x2="-33.02" y2="58.42" width="0.1524" layer="91"/>
@@
 </segment>
 <segment>
-<pinref part="U$1" gate="RJ45" pin="GND@2"/>
 <pinref part="SUPPLY9" gate="G$1" pin="RTN"/>
 <wire x1="-162.56" y1="238.76" x2="-162.56" y2="236.22" width="0.1524" layer="91"/>
@@
 <wire x1="-154.94" y1="236.22" x2="-154.94" y2="269.24" width="0.1524" layer="91"/>
 <wire x1="-154.94" y1="269.24" x2="-162.56" y2="269.24" width="0.1524" layer="91"/>
-<pinref part="U$1" gate="RJ45" pin="GND@0"/>
 <wire x1="-162.56" y1="269.24" x2="-162.56" y2="266.7" width="0.1524" layer="91"/>
-</segment>
-</net>
-<net name="N$20" class="0">
+<pinref part="X1" gate="G$1" pin="GND@0"/>
+<pinref part="X1" gate="G$1" pin="GND@2"/>
+</segment>
+</net>
+<net name="U4_SS" class="0">
 <segment>
 <pinref part="C37" gate="G$1" pin="1"/>
@@
 </segment>
 </net>
-<net name="N$30" class="0">
+<net name="INTVCC" class="0">
 <segment>
 <pinref part="D6" gate="G$1" pin="C"/>
@@
 <wire x1="-165.1" y1="210.82" x2="-167.64" y2="210.82" width="0.1524" layer="91"/>
 <junction x="-167.64" y="210.82"/>
-<pinref part="U$1" gate="RJ45" pin="POE+@4"/>
-<pinref part="U$1" gate="RJ45" pin="POE+@5"/>
+<pinref part="X1" gate="G$1" pin="POE+@4"/>
+<pinref part="X1" gate="G$1" pin="POE+@5"/>
 </segment>
 </net>
@@
 <wire x1="185.42" y1="175.26" x2="185.42" y2="172.72" width="0.1524" layer="91"/>
 <pinref part="GND8" gate="1" pin="GNDA"/>
-<pinref part="U$1" gate="LED2" pin="C"/>
+<pinref part="D1" gate="G$1" pin="C"/>
 </segment>
 <segment>
 <wire x1="195.58" y1="175.26" x2="195.58" y2="172.72" width="0.1524" layer="91"/>
 <pinref part="GND9" gate="1" pin="GNDA"/>
-<pinref part="U$1" gate="LED1" pin="C"/>
+<pinref part="D2" gate="G$1" pin="C"/>
 </segment>
 <segment>
@@
 <pinref part="R4" gate="G$1" pin="2"/>
 <wire x1="185.42" y1="185.42" x2="185.42" y2="182.88" width="0.1524" layer="91"/>
-<pinref part="U$1" gate="LED2" pin="A"/>
+<pinref part="D1" gate="G$1" pin="A"/>
 </segment>
 </net>
@@
 <pinref part="R3" gate="G$1" pin="1"/>
 <wire x1="195.58" y1="185.42" x2="195.58" y2="182.88" width="0.1524" layer="91"/>
-<pinref part="U$1" gate="LED1" pin="A"/>
+<pinref part="D2" gate="G$1" pin="A"/>
 </segment>
 </net>
@@
 </segment>
 </net>
-<net name="N$9" class="0">
+<net name="U5_CDB" class="0">
 <segment>
 <pinref part="R38" gate="1" pin="2"/>

Commit message: Small fix to PoElli-Nucleo
Parts:
- removed TP1: TEST_POINT-5000, ELL-i-Passives:TEST_POINT-5000
- SW1, SW2: value (none) -> A6H2101
Connections:
- net N$46 renamed VCAP
- removed net ETH_MUX: TP1.P$1
- net RTN: no longer X1.GND@0, X1.GND@2
- net SGND: now also X1.GND@0, X1.GND@2
Other:
- moved on the sheet: SW1
