File: PoElli/PoElli-Nucleo.sch (EAGLE design)
At the start: 120 parts, among them CN10 NUCLEO-CN10, CN7 NUCLEO-CN10, J3 M022.54MM, J4 M022.54MM, Q3 FDMC2674HANDSOLDERING, Q4 IRFL4310, SW1 A6H2101, SW2 A6H2101, T1 Coilcraft 230NL, T2 FLYBACK750311689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

Commit message: PoElli 0.4 Schema, tentative layout
Parts:
- removed C14: 100nF, ELL-i-Passives:C0402
- removed C23: 220uF, ELL-i-Passives:CPOLE
- removed C29: 1uF, ELL-i-Passives:C0805
- removed CN10, CN7: NUCLEO-CN10, ELL-i-Boards:NUCLEO-CN10
- removed NUCLEO: NUCLEO-SHIELD-OUTLINE-EXTENDED, ELL-i-Boards:NUCLEO-SHIELD-OUTLINE-EXTENDED
- removed R38: OPEN, SparkFun-Passives:SOLDERJUMPERNO
- removed SW1, SW2: A6H2101, SparkFun-Electromechanical:SW_DIP-2-SMT-HALFSIZE
- removed T2: FLYBACK750311689, ELL-i-Transformers:FLYBACK750311689
- added SJ1, SJ2, SJ3, SJ4: SOLDERJUMPERNO, SparkFun-Passives:SOLDERJUMPERNO
- added U$1: FLYBACK-3_OUTPUTS_749119350, ELL-i-Transformers:FLYBACK-3_OUTPUTS_749119350
- added U$2: NUCLEO-SHIELD-20PIN, ELL-i-Boards:NUCLEO-SHIELD-20PIN
- C1, C12, C19, C2, C36, C37, C38, C39: device ELL-i-Passives:C0402 -> ELL-i-Passives:C0805-A
- C13, C22, C42: device ELL-i-Passives:C0603 -> ELL-i-Passives:C0805-A
- C24, C25, C26, C27: value 10nF -> 10nF 100V; device ELL-i-Passives:C0603 -> ELL-i-Passives:C0805-A
- C28, C48: value 1nF -> 1nF 2kV
- C30: value 4u7 -> 4u7 25 V; device ELL-i-Passives:C0805 -> ELL-i-Passives:C0805-A
- C31: value 1nF -> 1nF 2kV; device ELL-i-Passives:C1210 -> ELL-i-Passives:C1206-A
- C32: device ELL-i-Passives:CPOLE -> ELL-i-Passives:C1206-A
- C33: value 150pF NP -> 150pF 200V NP; device ELL-i-Passives:C0805 -> ELL-i-Passives:C0805-A
- C34, C40: value 1nF -> 10nF 100V; device ELL-i-Passives:C0603 -> ELL-i-Passives:C0402-B
- C35, C41: value 100nF -> 100nF 100V; device ELL-i-Passives:C0805 -> ELL-i-Passives:C0805-A
- C4: value 47pF -> 100nF; device ELL-i-Passives:C0402 -> ELL-i-Passives:C0805-A
- C43, C44, C45, C46, C47: device ELL-i-Passives:C0805 -> ELL-i-Passives:C1206-A
- C5, C6, C7: value 1nF -> 100nF; device ELL-i-Passives:C0402 -> ELL-i-Passives:C0805-A
- C8, C9: device ELL-i-Passives:C0402 -> ELL-i-Passives:C0402-B
- D2: value YELLOW -> GREEN
- Q4: value IRFL4310 -> FDMC2674HANDSOLDERING; device ELL-i-DIscreteSemi:IRFL4310 -> ELL-i-DIscreteSemi:FDMC2674HANDSOLDERING
- R12, R13, R14, R6, R8, R9: device ELL-i-Passives:R0402 -> ELL-i-Passives:R0805-A
- R15, R18, R19, R20, R21, R24, R28, R30, R31, R33, R34, R35, R36: device ELL-i-Passives:R0603 -> ELL-i-Passives:R0805-A
- R27: device ELL-i-Passives:R0805 -> ELL-i-Passives:R0805-A
- R3, R4: value 180 -> 220; device ELL-i-Passives:R0402 -> ELL-i-Passives:R0805-A
- X1: value POE-TP-SHIELDED-RJ45-MOLEX-85502-5008 -> POE-TP-SHIELDED-LEDSTE1888250; device ELL-i-Connectors:POE-TP-SHIELDED-RJ45-MOLEX-85502-5008 -> ELL-i-Connectors:POE-TP-SHIELDED-LEDSTE1888250
Connections:
- removed net UNREG_6V+: C22.2, D4.A, T2.SEC+
- new net TRAFO_OUT: C22.2, D4.A, U$1.SEC1+, U$1.SEC2+, U$1.SEC3+
- net +3V3: now also U$2CN7.3V3_12, U$2CN7.3V3_16; no longer CN7.PA12_12, CN7.PB12_16
- net ETH_INT: now also SJ1.1, SJ2.1; no longer SW2.3, SW2.4
- net ETH_MISO: now also U$2CN10.27_PB4; no longer CN10.27_PB4
- net ETH_MOSI: now also U$2CN10.25_PB10; no longer CN10.25_PB10
- net ETH_SCK: now also U$2CN10.29_PB5; no longer CN10.29_PB5
- net ETH_SS: now also SJ3.1, SJ4.1; no longer SW1.3, SW1.4
- net GNDA: now also U$1.SEC1-, U$1.SEC2-, U$1.SEC3-, U$2CN7.GND_22; no longer C14.2, C23.-, CN7.PB2_22, T2.SEC-
- net N$1: now also X1RJ45.TX-@2; no longer X1.TX-@2
- net N$11: now also SJ3.2, U$2CN7.1_PC10; no longer CN7.1_PC9, SW1.2
- net N$12: now also SJ4.2, U$2CN7.3_PC12; no longer CN7.3_PB8, SW1.1
- net N$13: now also SJ2.2, U$2CN7.PC11_2; no longer CN7.PC8_2, SW2.1
- net N$14: now also SJ1.2, U$2CN7.PD2_4; no longer CN7.PC6_4, SW2.2
- net N$2: now also X1RJ45.TX+@1; no longer X1.TX+@1
- net N$28: now also U$1.PRI+; no longer T2.PRI+
- net N$29: now also U$1.AUX+; no longer T2.AUX+
- net N$3: now also X1RJ45.RX+@3; no longer X1.RX+@3
- net N$4: now also X1RJ45.RX-@6; no longer X1.RX-@6
- net POE_B+: now also X1RJ45.POE+@4, X1RJ45.POE+@5; no longer X1.POE+@4, X1.POE+@5
- net POE_B-: now also X1RJ45.POE-@7, X1RJ45.POE-@8; no longer X1.POE-@7, X1.POE-@8
- net RTN: now also C32.2, U$1.AUX-; no longer C29.2, C32.-, T2.AUX-
- net SGND: now also X1RJ45.GND@0, X1RJ45.GND@2; no longer X1.GND@0, X1.GND@2
- net U4_SS: no longer R38.1
- net U5_CDB: no longer R38.2
- net VCAP: no longer C14.1
- net VDD: now also C32.1, U$1.PRI-; no longer C29.1, C32.+, T2.PRI-
- net VIN: now also U$2CN7.VIN_24; no longer C23.+, CN7.PB1_24
Other:
- note added: "10 nF to simplify BoM"
- note added: "47 uF elco replaced with 10uF ceramic"
- note added: "Add reverse voltage prot?"
- note added: "Add zener ~8 V"
- note added: "Both leds same color to simplify BoM?"
- note added: "C8, C9 0402 for placement as close as possible to U6 pins"
- note added: "Calculate voltage ripple"
- note added: "D3, D6, D11 same diodes"
- note added: "Elco removed"
- note added: "R3, R4 same value as R27 to simplify BoM"
- note added: "R31, R33, C37, C38 values?"
- note added: "Removed 100nF"
- note added: "Replace with bridge?"
- note added: "SGND connection?"
- note added: "Same as Q3?"
- note added: "Same zener as load"
- note added: "Switches to solder bridges to save cost"
- note added: "TODO: replace package"
- note added: "Values?"
- note removed: "10V H6.2mm"
- note removed: "200V"
- note removed: "25V"
- note removed: "2kV"
- note removed: "R38 solder bridge is a potential alternative to R25, D11 and D13. To be tested."
- note removed: "XMK-8788K5-BX1X 1.5A Offset mounted connector Assembly upside down"
- moved on the sheet: C12, C28, C48
