File: PoElli/PoElli-Nucleo.sch (EAGLE design)
At the start: 107 parts, among them J3 M022.54MM, J4 M022.54MM, Q3 FDMC2674HANDSOLDERING, Q4 FDMC2674HANDSOLDERING, T1 Coilcraft 230NL, T2 FLYBACK-3_OUTPUTS_749119350, U4 LT3748, U5 TPS2378, U6 ENC424J600, X1 POE-TP-SHIELDED-LEDSTE1888250, Y1 25 MHz

Commit message: Fix SPI pin order
Connections:
- net ETH_MOSI: now also U$2CN10.29_PB5; no longer U$2CN10.25_PB10
- net ETH_SCK: now also U$2CN10.31_PB3; no longer U$2CN10.29_PB5
Changed lines of the file:
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@@
 <wire x1="302.26" y1="276.86" x2="215.9" y2="276.86" width="0.1524" layer="91"/>
 <pinref part="U6" gate="ENC424J600" pin="SCK/AL"/>
-<wire x1="307.34" y1="198.12" x2="302.26" y2="198.12" width="0.1524" layer="91"/>
-<wire x1="302.26" y1="198.12" x2="302.26" y2="276.86" width="0.1524" layer="91"/>
-<pinref part="U$2" gate="CN10" pin="29_PB5"/>
+<wire x1="302.26" y1="195.58" x2="302.26" y2="276.86" width="0.1524" layer="91"/>
+<pinref part="U$2" gate="CN10" pin="31_PB3"/>
+<wire x1="307.34" y1="195.58" x2="302.26" y2="195.58" width="0.1524" layer="91"/>
 </segment>
 <segment>
@@
 <wire x1="299.72" y1="274.32" x2="215.9" y2="274.32" width="0.1524" layer="91"/>
 <pinref part="U6" gate="ENC424J600" pin="SO/WR/EN"/>
+<pinref part="U$2" gate="CN10" pin="27_PB4"/>
+<wire x1="299.72" y1="200.66" x2="299.72" y2="274.32" width="0.1524" layer="91"/>
 <wire x1="307.34" y1="200.66" x2="299.72" y2="200.66" width="0.1524" layer="91"/>
-<wire x1="299.72" y1="200.66" x2="299.72" y2="274.32" width="0.1524" layer="91"/>
-<pinref part="U$2" gate="CN10" pin="27_PB4"/>
 </segment>
 <segment>
@@
 <wire x1="297.18" y1="271.78" x2="215.9" y2="271.78" width="0.1524" layer="91"/>
 <pinref part="U6" gate="ENC424J600" pin="SI/RD/!RW"/>
-<wire x1="307.34" y1="203.2" x2="297.18" y2="203.2" width="0.1524" layer="91"/>
-<wire x1="297.18" y1="203.2" x2="297.18" y2="271.78" width="0.1524" layer="91"/>
-<pinref part="U$2" gate="CN10" pin="25_PB10"/>
+<wire x1="297.18" y1="198.12" x2="297.18" y2="271.78" width="0.1524" layer="91"/>
+<pinref part="U$2" gate="CN10" pin="29_PB5"/>
+<wire x1="307.34" y1="198.12" x2="297.18" y2="198.12" width="0.1524" layer="91"/>
 </segment>
 <segment>

Commit message: Component placement complete
Parts:
- removed TP18: TEST_POINT-5000, ELL-i-Passives:TEST_POINT-5000
- added D10: MMSZ4694, ELL-i-DIscreteSemi:MMSZ4XXX
- added FID1, FID2, FID3: FIDUCIAL1X2, SparkFun-Aesthetics:FIDUCIAL1X2
- D13: value 18V -> MMSZ4694 (8V2); device ELL-i-DIscreteSemi:DIODE-ZENER-SOD-123 -> ELL-i-DIscreteSemi:MMSZ4XXX
- D18, D19: value B2100 -> SMD1200PL; device ELL-i-DIscreteSemi:DIODE-SCHOTTKYB2100 -> ELL-i-DIscreteSemi:SMD1XXPL
- D3: value BAV20WS -> SMD1200PL; device ELL-i-DIscreteSemi:BAV20WS -> ELL-i-DIscreteSemi:SMD1XXPL
- D6: value BAS70J -> SMD1200PL; device ELL-i-DIscreteSemi:BAS70J -> ELL-i-DIscreteSemi:SMD1XXPL
- TP5: value TEST_POINT-5000 -> TEST_POINT-5021; device ELL-i-Passives:TEST_POINT-5000 -> ELL-i-Passives:TEST_POINT-5021
- renumbered TP7 to 3V3
Connections:
- removed net N$36: D1.A, R4.2
- removed net N$38: D2.A, R3.1
- new net LEDA: D2.A, R3.1, X1LED1.A
- new net LEDB: D1.A, R4.2, X1LED2.A
- net GNDA: now also D10.A, X1LED1.C, X1LED2.C
- net SGND: no longer TP18.P$1
- net VIN: now also D10.C
Other:
- note added: "Added zener ~8 V"
- note added: "FIDUCIALS AT EDGES"
- note added: "Fixed pin order, verify"
- note added: "Replaced to simplify BOM"
- note removed: "Add zener ~8 V"
- moved on the sheet: X1LED1, X1LED2

Commit message: Copper layers, complete, DRC ok. Silkscreen has to be adjusted.
Parts:
- X1: value POE-TP-SHIELDED-LEDSTE1888250 -> POE-TP-SHIELDED-LEDSTE1888250-A; device ELL-i-Connectors:POE-TP-SHIELDED-LEDSTE1888250 -> ELL-i-Connectors:POE-TP-SHIELDED-LEDSTE1888250-A
- renumbered TP2 to SS, TP6 to INT
Changed lines of the file:
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@@
 <grid distance="0.1" unitdist="inch" unit="inch" style="lines" multiple="1" display="no" altdistance="0.01" altunitdist="inch" altunit="inch"/>
 <layers>
-<layer number="1" name="Top" color="4" fill="1" visible="yes" active="no"/>
-<layer number="2" name="Route2" color="4" fill="15" visible="yes" active="no"/>
-<layer number="3" name="Route3" color="4" fill="3" visible="yes" active="no"/>
-<layer number="14" name="Route14" color="1" fill="6" visible="yes" active="no"/>
-<layer number="15" name="Route15" color="1" fill="15" visible="yes" active="no"/>
-<layer number="16" name="Bottom" color="1" fill="1" visible="yes" active="no"/>
-<layer number="17" name="Pads" color="2" fill="1" visible="yes" active="no"/>
-<layer number="18" name="Vias" color="2" fill="1" visible="yes" active="no"/>
-<layer number="19" name="Unrouted" color="6" fill="1" visible="yes" active="no"/>
-<layer number="20" name="Dimension" color="15" fill="1" visible="yes" active="no"/>
-<layer number="21" name="tPlace" color="11" fill="1" visible="yes" active="no"/>
-<layer number="22" name="bPlace" color="7" fill="1" visible="yes" active="no"/>
-<layer number="23" name="tOrigins" color="15" fill="1" visible="yes" active="no"/>
-<layer number="24" name="bOrigins" color="15" fill="1" visible="yes" active="no"/>
-<layer number="25" name="tNames" color="11" fill="1" visible="yes" active="no"/>
-<layer number="26" name="bNames" color="7" fill="1" visible="yes" active="no"/>
-<layer number="27" name="tValues" color="7" fill="1" visible="yes" active="no"/>
-<layer number="28" name="bValues" color="7" fill="1" visible="yes" active="no"/>
+<layer number="1" name="Top" color="4" fill="1" visible="no" active="no"/>
+<layer number="2" name="Route2" color="2" fill="1" visible="no" active="no"/>
+<layer number="3" name="Route3" color="4" fill="3" visible="no" active="no"/>
+<layer number="14" name="Route14" color="1" fill="6" visible="no" active="no"/>
+<layer number="15" name="Route15" color="10" fill="15" visible="no" active="no"/>
+<layer number="16" name="Bottom" color="1" fill="1" visible="no" active="no"/>
+<layer number="17" name="Pads" color="2" fill="1" visible="no" active="no"/>
+<layer number="18" name="Vias" color="2" fill="1" visible="no" active="no"/>
+<layer number="19" name="Unrouted" color="6" fill="1" visible="no" active="no"/>
+<layer number="20" name="Dimension" color="15" fill="1" visible="no" active="no"/>
+<layer number="21" name="tPlace" color="11" fill="1" visible="no" active="no"/>
+<layer number="22" name="bPlace" color="7" fill="1" visible="no" active="no"/>
+<layer number="23" name="tOrigins" color="15" fill="1" visible="no" active="no"/>
+<layer number="24" name="bOrigins" color="15" fill="1" visible="no" active="no"/>
+<layer number="25" name="tNames" color="11" fill="1" visible="no" active="no"/>
+<layer number="26" name="bNames" color="7" fill="1" visible="no" active="no"/>
+<layer number="27" name="tValues" color="7" fill="1" visible="no" active="no"/>
+<layer number="28" name="bValues" color="7" fill="1" visible="no" active="no"/>
 <layer number="29" name="tStop" color="7" fill="3" visible="no" active="no"/>
 <layer number="30" name="bStop" color="7" fill="6" visible="no" active="no"/>
@@
 <layer number="35" name="tGlue" color="7" fill="4" visible="no" active="no"/>
 <layer number="36" name="bGlue" color="7" fill="5" visible="no" active="no"/>
-<layer number="37" name="tTest" color="7" fill="1" visible="yes" active="no"/>
-<layer number="38" name="bTest" color="7" fill="1" visible="yes" active="no"/>
+<layer number="37" name="tTest" color="7" fill="1" visible="no" active="no"/>
+<layer number="38" name="bTest" color="7" fill="1" visible="no" active="no"/>
 <layer number="39" name="tKeepout" color="4" fill="11" visible="no" active="no"/>
 <layer number="40" name="bKeepout" color="1" fill="11" visible="no" active="no"/>
 <layer number="41" name="tRestrict" color="4" fill="2" visible="no" active="no"/>
-<layer number="42" name="bRestrict" color="1" fill="10" visible="no" active="no"/>
+<layer number="42" name="bRestrict" color="1" fill="15" visible="no" active="no"/>
 <layer number="43" name="vRestrict" color="2" fill="10" visible="no" active="no"/>
 <layer number="44" name="Drills" color="7" fill="1" visible="no" active="no"/>
 <layer number="45" name="Holes" color="7" fill="1" visible="no" active="no"/>
-<layer number="46" name="Milling" color="3" fill="1" visible="yes" active="no"/>
-<layer number="47" name="Measures" color="8" fill="1" visible="yes" active="no"/>
-<layer number="48" name="Document" color="7" fill="1" visible="yes" active="no"/>
-<layer number="49" name="Reference" color="7" fill="1" visible="yes" active="no"/>
-<layer number="50" name="dxf" color="7" fill="1" visible="yes" active="no"/>
-<layer number="51" name="tDocu" color="1" fill="1" visible="yes" active="no"/>
-<layer number="52" name="bDocu" color="7" fill="1" visible="yes" active="no"/>
-<layer number="53" name="tGND_GNDA" color="7" fill="9" visible="yes" active="no"/>
-<layer number="54" name="bGND_GNDA" color="1" fill="9" visible="yes" active="no"/>
-<layer number="56" name="wert" color="7" fill="1" visible="yes" active="no"/>
-<layer number="57" name="tCopper" color="7" fill="1" visible="yes" active="no"/>
-<layer number="58" name="bCopper" color="7" fill="1" visible="yes" active="no"/>
+<layer number="46" name="Milling" color="3" fill="1" visible="no" active="no"/>
+<layer number="47" name="Measures" color="8" fill="1" visible="no" active="no"/>
+<layer number="48" name="Document" color="7" fill="1" visible="no" active="no"/>
+<layer number="49" name="Reference" color="7" fill="1" visible="no" active="no"/>
+<layer number="50" name="dxf" color="7" fill="1" visible="no" active="no"/>
+<layer number="51" name="tDocu" color="1" fill="1" visible="no" active="no"/>
+<layer number="52" name="bDocu" color="7" fill="1" visible="no" active="no"/>
+<layer number="53" name="tGND_GNDA" color="7" fill="9" visible="no" active="no"/>
+<layer number="54" name="bGND_GNDA" color="1" fill="9" visible="no" active="no"/>
+<layer number="56" name="wert" color="7" fill="1" visible="no" active="no"/>
+<layer number="57" name="tCopper" color="7" fill="1" visible="no" active="no"/>
+<layer number="58" name="bCopper" color="7" fill="1" visible="no" active="no"/>
 <layer number="91" name="Nets" color="2" fill="1" visible="yes" active="yes"/>
 <layer number="92" name="Busses" color="1" fill="1" visible="yes" active="yes"/>
@@
 <part name="R15" library="ELL-i-Passives" deviceset="R" device="0603-B" value="10R"/>
 <part name="C22" library="ELL-i-Passives" deviceset="C" device="0603-B" value="470pF"/>
-<part name="TP2" library="ELL-i-Passives" deviceset="TEST_POINT" device="-5021" value=""/>
+<part name="SS" library="ELL-i-Passives" deviceset="TEST_POINT" device="-5021" value=""/>
 <part name="TP3" library="ELL-i-Passives" deviceset="TEST_POINT" device="-5021" value=""/>
 <part name="TP4" library="ELL-i-Passives" deviceset="TEST_POINT" device="-5021" value=""/>
 <part name="TP5" library="ELL-i-Passives" deviceset="TEST_POINT" device="-5021" value="TEST_POINT-5021"/>
-<part name="TP6" library="ELL-i-Passives" deviceset="TEST_POINT" device="-5000" value=""/>
+<part name="INT" library="ELL-i-Passives" deviceset="TEST_POINT" device="-5000" value=""/>
 <part name="3V3" library="ELL-i-Passives" deviceset="TEST_POINT" device="-5000" value=""/>
 <part name="TP9" library="ELL-i-Passives" deviceset="TEST_POINT" device="-5000" value=""/>
@@
 <part name="GND1" library="supply1" deviceset="GNDA" device=""/>
 <part name="U$2" library="ELL-i-Boards" deviceset="NUCLEO-SHIELD" device="-20PIN"/>
-<part name="X1" library="ELL-i-Connectors" deviceset="POE-TP-SHIELDED-LEDS" device="TE1888250"/>
+<part name="X1" library="ELL-i-Connectors" deviceset="POE-TP-SHIELDED-LEDS" device="TE1888250-A" value="POE-TP-SHIELDED-LEDSTE1888250-A"/>
 <part name="C4" library="ELL-i-Passives" deviceset="C" device="0603-B" value="100nF"/>
 <part name="B1" library="ELL-i-DIscreteSemi" deviceset="BRIDGE-RECTIFIER" device=""/>
@@
 <instance part="R15" gate="G$1" x="-38.1" y="208.28"/>
 <instance part="C22" gate="G$1" x="-48.26" y="208.28" rot="MR90"/>
-<instance part="TP2" gate="TP$1" x="274.32" y="205.74" rot="R90"/>
+<instance part="SS" gate="TP$1" x="274.32" y="205.74" rot="R90"/>
 <instance part="TP3" gate="TP$1" x="274.32" y="198.12" rot="R90"/>
 <instance part="TP4" gate="TP$1" x="274.32" y="190.5" rot="R90"/>
 <instance part="TP5" gate="TP$1" x="274.32" y="182.88" rot="R90"/>
-<instance part="TP6" gate="TP$1" x="274.32" y="175.26" rot="R90"/>
+<instance part="INT" gate="TP$1" x="274.32" y="175.26" rot="R90"/>
 <instance part="3V3" gate="TP$1" x="274.32" y="167.64" rot="R90"/>
 <instance part="TP9" gate="TP$1" x="274.32" y="160.02" rot="R90"/>
@@
 </segment>
 <segment>
-<pinref part="TP6" gate="TP$1" pin="P$1"/>
+<pinref part="INT" gate="TP$1" pin="P$1"/>
 <wire x1="261.62" y1="175.26" x2="271.78" y2="175.26" width="0.1524" layer="91"/>
 <label x="261.62" y="175.26" size="1.778" layer="95" rot="R180" xref="yes"/>
@@
 </segment>
 <segment>
-<pinref part="TP2" gate="TP$1" pin="P$1"/>
+<pinref part="SS" gate="TP$1" pin="P$1"/>
 <wire x1="271.78" y1="205.74" x2="261.62" y2="205.74" width="0.1524" layer="91"/>
 <label x="261.62" y="205.74" size="1.778" layer="95" rot="R180" xref="yes"/>

Commit message: Silkscreen ok
Parts:
- 3V3: value TEST_POINT-5000 -> 3V3
- C40: device ELL-i-Passives:C0402-B -> ELL-i-Passives:C0603-B
- D1: value GREEN -> LINK
- D2: value GREEN -> ACT
- MISO: value TEST_POINT-5021 -> MISO
- SS: value TEST_POINT-5021 -> SS
- TP3: value TEST_POINT-5021 -> SCK
- TP4: value TEST_POINT-5021 -> MOSI
- TP9: value TEST_POINT-5000 -> GND
- renumbered TP5 to MISO
Changed lines of the file:
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@@
 <part name="C24" library="ELL-i-Passives" deviceset="C" device="0603-B" value="10nF 100V"/>
 <part name="J4" library="SparkFun-Connectors" deviceset="M02" device="2.54MM_SCREWTERM" value="M022.54MM"/>
-<part name="C40" library="ELL-i-Passives" deviceset="C" device="0402-B" value="10nF 100V"/>
+<part name="C40" library="ELL-i-Passives" deviceset="C" device="0603-B" value="10nF 100V"/>
 <part name="C41" library="ELL-i-Passives" deviceset="C" device="0603-B" value="100nF 100V"/>
 <part name="C42" library="ELL-i-Passives" deviceset="C" device="0603-B" value="10nF"/>
@@
 <part name="R15" library="ELL-i-Passives" deviceset="R" device="0603-B" value="10R"/>
 <part name="C22" library="ELL-i-Passives" deviceset="C" device="0603-B" value="470pF"/>
-<part name="SS" library="ELL-i-Passives" deviceset="TEST_POINT" device="-5021" value=""/>
-<part name="TP3" library="ELL-i-Passives" deviceset="TEST_POINT" device="-5021" value=""/>
-<part name="TP4" library="ELL-i-Passives" deviceset="TEST_POINT" device="-5021" value=""/>
-<part name="TP5" library="ELL-i-Passives" deviceset="TEST_POINT" device="-5021" value="TEST_POINT-5021"/>
-<part name="INT" library="ELL-i-Passives" deviceset="TEST_POINT" device="-5000" value=""/>
-<part name="3V3" library="ELL-i-Passives" deviceset="TEST_POINT" device="-5000" value=""/>
-<part name="TP9" library="ELL-i-Passives" deviceset="TEST_POINT" device="-5000" value=""/>
+<part name="SS" library="ELL-i-Passives" deviceset="TEST_POINT" device="-5021" value="SS"/>
+<part name="TP3" library="ELL-i-Passives" deviceset="TEST_POINT" device="-5021" value="SCK"/>
+<part name="TP4" library="ELL-i-Passives" deviceset="TEST_POINT" device="-5021" value="MOSI"/>
+<part name="MISO" library="ELL-i-Passives" deviceset="TEST_POINT" device="-5021" value="MISO"/>
+<part name="INT" library="ELL-i-Passives" deviceset="TEST_POINT" device="-5000" value="TEST_POINT-5000"/>
+<part name="3V3" library="ELL-i-Passives" deviceset="TEST_POINT" device="-5000" value="3V3"/>
+<part name="TP9" library="ELL-i-Passives" deviceset="TEST_POINT" device="-5000" value="GND"/>
 <part name="U$6" library="SparkFun-Aesthetics" deviceset="FRAME-A4L" device=""/>
 <part name="GND3" library="supply1" deviceset="GNDA" device=""/>
@@
 <part name="+3V3" library="supply1" deviceset="+3V3" device=""/>
 <part name="+3V4" library="supply1" deviceset="+3V3" device=""/>
-<part name="D1" library="SparkFun-LED" deviceset="LED-GREEN" device="0603" value="GREEN"/>
-<part name="D2" library="SparkFun-LED" deviceset="LED-YELLOW" device="0603" value="GREEN"/>
+<part name="D1" library="SparkFun-LED" deviceset="LED-GREEN" device="0603" value="LINK"/>
+<part name="D2" library="SparkFun-LED" deviceset="LED-YELLOW" device="0603" value="ACT"/>
 <part name="SJ1" library="SparkFun-Passives" deviceset="SOLDERJUMPER" device="NO"/>
 <part name="SJ2" library="SparkFun-Passives" deviceset="SOLDERJUMPER" device="NO"/>
@@
 <instance part="TP3" gate="TP$1" x="274.32" y="198.12" rot="R90"/>
 <instance part="TP4" gate="TP$1" x="274.32" y="190.5" rot="R90"/>
-<instance part="TP5" gate="TP$1" x="274.32" y="182.88" rot="R90"/>
+<instance part="MISO" gate="TP$1" x="274.32" y="182.88" rot="R90"/>
 <instance part="INT" gate="TP$1" x="274.32" y="175.26" rot="R90"/>
 <instance part="3V3" gate="TP$1" x="274.32" y="167.64" rot="R90"/>
@@
 </segment>
 <segment>
-<pinref part="TP5" gate="TP$1" pin="P$1"/>
+<pinref part="MISO" gate="TP$1" pin="P$1"/>
 <wire x1="271.78" y1="182.88" x2="261.62" y2="182.88" width="0.1524" layer="91"/>
 <label x="261.62" y="182.88" size="1.778" layer="95" rot="R180" xref="yes"/>
