File: PoElli/PoElli-Nucleo.brd (EAGLE design)
At the start: 160 x 100 mm, 112 parts, among them J3 M022.54MM, J4 M022.54MM, Q3 FDMC2674HANDSOLDERING, Q4 FDMC2674HANDSOLDERING, T1 Coilcraft 230NL, T2 FLYBACK-3_OUTPUTS_749119350, U4 LT3748, U5 TPS2378, U6 ENC424J600, X1 POE-TP-SHIELDED-LEDSTE1888250, Y1 25 MHz

Commit message: Component placement almost ready
Parts:
- removed C31: 1nF 2kV, ELL-i-Passives:SMD1206-A
- removed C36: 47p, ELL-i-Passives:SMD0805-A
- removed D11: BAS70J, ELL-i-DIscreteSemi:SOD-323
- removed R25: 100K, ELL-i-Passives:SMD0805-A
- removed R30: 0R, ELL-i-Passives:SMD0805-A
- C1, C11, C12, C13, C15, C2, C21, C22, C24, C25, C26, C27, C3, C30, C33, C34, C35, C37, C38, C39, C4, C41, C42, C5, C6, C7, R12, R13, R15, R18, R19, R20, R21, R22, R23, R24, R26, R27, R28, R29, R33, R35, R36, R6, R8, R9: device ELL-i-Passives:SMD0805-A -> ELL-i-Passives:SMD0603-B
- FB2, FB3, FB5: device ELL-i-Passives:SMD0805-A -> ELL-i-Passives:SMD0603-A
- R32: value 0R03 -> 0R10; device ELL-i-Passives:SMD0805-A -> ELL-i-Passives:SMD0603-B
- moved R33 188.1 mm to (102.7, 50.4), turned to 180 degrees
- moved C38 183.8 mm to (105.5, 50.4)
- moved C48 181.3 mm to (63.0, 55.5), turned to 90 degrees
- moved D6 181.1 mm to (104.4, 54.5), turned to 90 degrees
- moved C39 171.2 mm to (98.8, 55.0), turned to 90 degrees
- moved D3 162.9 mm to (90.9, 50.6), turned to 90 degrees
- moved R27 159.0 mm to (92.9, 46.4)
- moved C30 152.9 mm to (99.8, 46.3)
- moved R16 152.4 mm to (87.5, 48.9), turned to 180 degrees
- moved C33 150.2 mm to (92.5, 49.8), turned to 270 degrees
- moved C21 149.6 mm to (88.0, 51.1)
- moved FB1 120.4 mm to (55.1, 55.7), turned to 90 degrees
- moved R6 118.0 mm to (64.8, 67.2)
- moved C28 44.5 mm to (89.5, 64.8), turned to 90 degrees
- moved C10 35.0 mm to (80.4, 30.4), turned to 270 degrees
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Connections:
- removed net N$27: Q3.1, Q3.2, Q3.3, R30.P$1, R32.P$1
- removed net N$9: C10.P$1, R20.P$1, R21.P$1
- removed net U5_CDB: D11.C, D13.C, Q4.4, R25.P$2, U5.6
- net GNDA: now also C10.P$2
- net N$26: now also Q3.1, Q3.2, Q3.3, R32.P$1; no longer C36.P$1, R30.P$2
- net N$5: now also C10.P$1, R20.P$1, R21.P$1; no longer C31.P$1
- net RTN: no longer C36.P$2
- net SGND: no longer C10.P$2, C31.P$2
- net U4_EN: now also D13.C, Q4.4, U5.6; no longer D11.A
- net VDD: no longer R25.P$1
Routing:
- net POE_A-: track 0.00 -> 29.0 mm
- net POE_A+: track 0.00 -> 21.6 mm
- net N$5: track 0.00 -> 20.3 mm
- net POE_B-: track 0.00 -> 16.5 mm
- net POE_B+: track 0.00 -> 14.5 mm
- net N$37: track 0.00 -> 7.30 mm
- net N$47: track 0.00 -> 5.40 mm
- net N$45: track 0.00 -> 2.38 mm
- net ENC-3V3: track 0.00 -> 2.29 mm
- net N$52: track 0.00 -> 1.47 mm
- net N$48: track 0.00 -> 1.38 mm
- net N$51: track 0.00 -> 1.32 mm
- net N$50: track 0.00 -> 1.32 mm

Commit message: DC/DC layout except planes
Parts:
- C19, R31, R34, R5: device ELL-i-Passives:SMD0805-A -> ELL-i-Passives:SMD0603-B
- R3, R4: device ELL-i-Passives:SMD0805-A -> ELL-i-Passives:SMD0603-A
- moved SJ1 192.8 mm to (64.2, 49.4), turned to 270 degrees
- moved C40 192.5 mm to (102.2, 37.0)
- moved R34 187.9 mm to (98.2, 55.0), turned to 270 degrees
- moved R31 182.6 mm to (102.8, 50.0), turned to 180 degrees
- moved R4 180.4 mm to (57.4, 55.8), turned to 270 degrees
- moved R3 177.6 mm to (59.4, 55.8), turned to 90 degrees
- moved R14 176.7 mm to (59.5, 50.3), turned to 90 degrees
- moved TP4 151.2 mm to (32.5, 58.3)
- moved TP2 137.0 mm to (29.2, 62.8)
- moved TP3 137.0 mm to (24.1, 62.8)
- moved TP5 137.0 mm to (49.5, 62.8)
- moved TP6 137.0 mm to (44.5, 62.8)
- moved TP7 137.0 mm to (39.4, 62.8)
- moved TP9 137.0 mm to (34.3, 62.8)
- moved TP18 133.1 mm to (24.4, 58.5)
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Routing:
- net N$6: track 0.00 -> 22.1 mm
- net N$28: track 0.00 -> 21.4 mm
- net N$8: track 0.00 -> 21.3 mm
- net RTN: track 0.00 -> 17.1 mm
- net N$10: track 0.00 -> 15.9 mm
- net U4_EN: track 0.00 -> 14.8 mm
- net N$54: track 0.00 -> 14.6 mm, vias 0 -> 2
- net VDD: track 0.00 -> 14.6 mm
- net N$55: track 0.00 -> 13.3 mm
- net VSS: track 0.00 -> 12.5 mm
- net INTVCC: track 0.00 -> 12.5 mm
- net N$26: track 0.00 -> 12.5 mm
- net N$76: track 0.00 -> 11.0 mm
- net N$53: track 0.00 -> 9.52 mm
- net N$21: track 0.00 -> 9.06 mm
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Other:
- board size 160 x 100 mm -> 57.5 x 70 mm
- board text added: "-IN+ 48V 0A3"
- board text removed: "48V 0A3"
