File: Baselli/Baselli.sch (EAGLE design)
At the start: 76 parts, among them J2 DF12-ELLI-HEADER-TOP, J3 DF12-ELLI-RECEPTABLE-BOTTOM, J4 FTDI-SER-6-PP, J5 JTAG_PROG, Q1 IRLML2244, SW1 A6H-2101, U1 LCMXO2-256HC-4SG32, U2 STM32F051R, X1 8MHz NP, X2 32.768 kHz

Commit message: Fixups and renumbering in Baselli
Parts:
- removed J5: JTAG_PROG, ELL-i-Connectors:JTAG_PROG
- removed U2: STM32F051R, ELL-i-DigitalIC:STM32F051R
- removed X1: 8MHz NP, SparkFun-FreqCtrl:CRYSTAL_WITH_GND
- added J1: FTDI-SER-6-PP, ELL-i-Connectors:FTDI-SER-6-PP
- added Q2: IRLML2244, SparkFun-DiscreteSemi:MOSFET-PCHANNELIRLML2244
- added U4: LCMXO2-256HC-4SG32, ELL-i-DigitalIC:LCMXO2-256HC-4SG32
- C1: value 15 pF -> 33n
- C10: value 33n -> 1uF
- C11: value 15 pF -> 10nF
- C3: value 10nF -> 100nF
- C5: value 22pF -> 1uF
- C7: value 1uF -> 22pF
- C8: value 1uF -> 15 pF
- C9: value 100nF -> 15 pF
- D1: value WS2182B -> GREEN; device SparkFun-LED:WS2812B -> SparkFun-LED:LED-GREEN0603
- D2: value GREEN -> BAT60J; device SparkFun-LED:LED-GREEN0603 -> SparkFun-DiscreteSemi:DIODE-SCHOTTKY-BAT60J
- D5: value BAT60J -> WS2182B; device SparkFun-DiscreteSemi:DIODE-SCHOTTKY-BAT60J -> SparkFun-LED:WS2812B
- J4: value FTDI-SER-6-PP -> JTAG_PROG; device ELL-i-Connectors:FTDI-SER-6-PP -> ELL-i-Connectors:JTAG_PROG
- Q1: value IRLML2244 -> 8MHz NP; device SparkFun-DiscreteSemi:MOSFET-PCHANNELIRLML2244 -> SparkFun-FreqCtrl:CRYSTAL_WITH_GND
- R10: value 4K7 (NP) -> 2K2; device ELL-i-Passives:R0603 -> ELL-i-Passives:R0402
- R11: value 47K -> 180; device ELL-i-Passives:R0402 -> ELL-i-Passives:R0805
- R12: value NP -> 0
- R13: value 10k -> 180
- R17: value 0 -> 180
- R19, R21: value 180 -> 10K; device ELL-i-Passives:R0805 -> ELL-i-Passives:R0402
- R2: value 390R -> 10k
- R20: value 180 -> 4K7 (NP); device ELL-i-Passives:R0805 -> ELL-i-Passives:R0603
- R22: value NP -> 47K; device ELL-i-Passives:R0805 -> ELL-i-Passives:R0402
- R23: value 1k5 -> NP; device ELL-i-Passives:R0402 -> ELL-i-Passives:R0805
- R3: value 10k -> 390R
- R4: value 2K2 -> 1k5
- R5: value 2K2 -> 10k; device ELL-i-Passives:R0402 -> ELL-i-Passives:R0805
- R8: value 10K -> NP; device ELL-i-Passives:R0402 -> ELL-i-Passives:R0805
- R9: value 10K -> 2K2
- U1: value LCMXO2-256HC-4SG32 -> STM32F051R; device ELL-i-DigitalIC:LCMXO2-256HC-4SG32 -> ELL-i-DigitalIC:STM32F051R
- renumbered X2 to Y1
Connections:
- net +3V3: now also C2.1, C3.1, C5.1, D1.A, D2.C, J4.1, Q2.S, R10.1, R19.1, R22.1, U1PWR.VDD, U4PWR.VCC; no longer C7.1, C8.1, C9.1, D2.A, D5.C, J5.1, Q1.S, R11.1, R4.1, R5.1, U1PWR.VCC, U2PWR.VDD
- net +5V: now also D5.VDD; no longer D1.VDD
- net -RTS: now also C1.2; no longer C10.2
- net A0: now also U1PA.PA0-ADC_IN0; no longer U2PA.PA0-ADC_IN0
- net A1: now also U1PA.PA2-ADC_IN2; no longer U2PA.PA2-ADC_IN2
- net A2: now also U1PA.PA4-ADC_IN4; no longer U2PA.PA4-ADC_IN4
- net A3: now also U1PA.PA5-ADC_IN5; no longer U2PA.PA5-ADC_IN5
- net A4: now also R10.2, U1PB.PB9, U4ERB.SDA/PT12D; no longer R7.2, U1ERB.SDA/PT12D, U2PB.PB9
- net A5: now also R7.2, U1PB.PB6, U4ERB.SCL/PT12C; no longer R6.2, U1ERB.SCL/PT12C, U2PB.PB6
- net AREF: now also R5.2; no longer R13.1
- net BOOT0: now also R4.2, U1CTL.BOOT0; no longer R23.2, U2CTL.BOOT0
- net BOOT0TX: now also J1.TXD, R2.1; no longer J4.TXD, R3.2
- net CSSPIN: now also U1PC.PC12, U4ERB.CSSPIN/PB_2A...; no longer U1ERB.CSSPIN/PB_2A..., U2PC.PC12
- net D0: now also R2.2, U1PA.PA10; no longer R3.1, U2PA.PA10
- net D1: now also J1.RXD, U1PA.PA9; no longer J4.RXD, U2PA.PA9
- net D10: now also J4.6, U1PA.PA15, U4ERB.TDO; no longer J5.6, U1ERB.TDO, U2PA.PA15
- net D11: now also U1PB.PB5, U4ERB.SISPI/PB20D; no longer U1ERB.SISPI/PB20D, U2PB.PB5
- net D12: now also U1PA.PA6-ADC_IN6, U4ERB.SPISO/PB6D; no longer U1ERB.SPISO/PB6D, U2PA.PA6-ADC_IN6
- net D13: now also U1PB.PB3, U4ERB.MCLK/CCLK/PB6C; no longer U1ERB.MCLK/CCLK/PB6C, U2PB.PB3
- net D2: now also U1PDF.PD2; no longer U2PDF.PD2
- net D3: now also J1.-CTS, U1PA.PA11; no longer J4.-CTS, U2PA.PA11
- net D4: now also C1.1, J1.-RTS, U1PA.PA12; no longer C10.1, J4.-RTS, U2PA.PA12
- net D5: now also U1PB.PB1-ADC_IN9; no longer U2PB.PB1-ADC_IN9
- net D6: now also U1PA.PA3-ADC_IN3; no longer U2PA.PA3-ADC_IN3
- net D7: now also R15.2, SJ10.1; no longer R15.1, SJ14.1
- net D8: now also U1PB.PB7; no longer U2PB.PB7
- net D9: now also R14.2, SJ12.1; no longer R14.1, SJ9.1
- net DONE: now also SJ10.2, U4ERB.DONE/PT17D; no longer SJ14.2, U1ERB.DONE/PT17D
- net DOUT: now also D5.DOUT; no longer D1.DOUT
- net E0: now also R17.2, SJ8.1; no longer R18.2, SJ10.1
- net E1: now also R11.2, SJ13.1; no longer R19.2, SJ11.1
- net E10: now also U1PC.PC6; no longer U2PC.PC6
- net E11: now also U1PC.PC7; no longer U2PC.PC7
- net E12: now also R16.2, R9.2, SJ11.1; no longer R17.2, R5.2, SJ7.1
- net E13: now also R12.2, R6.2, SJ7.1; no longer R16.1, R4.2, SJ8.1
- net E14: now also U1PB.PB12; no longer U2PB.PB12
- net E15: now also U1PB.PB15; no longer U2PB.PB15
- net E16: now also U1PB.PB14; no longer U2PB.PB14
- net E17: now also U1PB.PB13; no longer U2PB.PB13
- net E18: now also U1PC.PC11; no longer U2PC.PC11
- net E19: now also U1PC.PC10; no longer U2PC.PC10
- net E2: now also R13.2, SJ9.1; no longer R20.2, SJ12.1
- net E3: now also R18.2, SJ14.1; no longer R21.2, SJ13.1
- net E4: now also U1PC.PC0-ADC_IN10; no longer U2PC.PC0-ADC_IN10
- net E5: now also U1PC.PC1-ADC_IN11; no longer U2PC.PC1-ADC_IN11
- net E6: now also U1PC.PC2-ADC_IN12; no longer U2PC.PC2-ADC_IN12
- net E7: now also U1PC.PC3-ADC_IN13; no longer U2PC.PC3-ADC_IN13
- net E8: now also U1PC.PC4-ADC_IN14; no longer U2PC.PC4-ADC_IN14
- net E9: now also U1PC.PC5-ADC_IN15; no longer U2PC.PC5-ADC_IN15
- net ETH_INT: now also U1PA.PA1-ADC_IN1; no longer U2PA.PA1-ADC_IN1
- net ETH_SS: now also U1PC.PC13; no longer U2PC.PC13
- net GNDI: now also C2.2, C3.2, C4.1, C5.2, C7.1, C8.1, C9.1, D5.VSS, J1.GND, J4.5, J4.9, Q1.GND@1, Q1.GND@2, R20.2, R21.1, R4.1, U1PWR.VSS, U4PWR.GND; no longer C1.1, C11.1, C4.2, C5.1, C7.2, C8.2, C9.2, D1.VSS, J4.GND, J5.5, J5.9, R10.2, R12.1, R8.1, U1PWR.GND, U2PWR.VSS, X1.GND@1, X1.GND@2
- net JTAGENB: now also Q2.D, R21.2, U4ERB.JTAGENB/PT15C; no longer Q1.D, R8.2, U1ERB.JTAGENB/PT15C
- net JTAGENB_MCU: now also U1PB.PB4; no longer U2PB.PB4
- net JTAGEN_GATE: now also J4.3, Q2.G, R22.2; no longer J5.3, Q1.G, R11.2
- net JTDI: now also J4.8, U1PC.PC9, U4ERB.TDI; no longer J5.8, U1ERB.TDI, U2PC.PC9
- net MCO: now also U1PA.PA8, U4IO.PR_5A/5C/5C/7A/10A; no longer U1IO.PR_5A/5C/5C/7A/10A, U2PA.PA8
- net N$1: now also SJ1.2, U4PWR.VCCIO0; no longer SJ4.2, U1PWR.VCCIO0
- net N$10: now also SJ13.2, U4IO.PB_4B/6D/9B/11B/13B; no longer SJ11.2, U1IO.PB_4B/6D/9B/11B/13B
- net N$12: now also SJ12.2, U4IO.PR_5B/5D/5D/7B/10B; no longer SJ9.2, U1IO.PR_5B/5D/5D/7B/10B
- net N$15: now also SJ9.2, U4IO.PB_4C/10C/11A/16A/20A; no longer SJ12.2, U1IO.PB_4C/10C/11A/16A/20A
- net N$16: now also SJ14.2, U4IO.PB_4D/10D/11B/16B/20B; no longer SJ13.2, U1IO.PB_4D/10D/11B/16B/20B
- net N$17: now also SJ11.2, U4IO.PL_5C/7A/9A/12A/17A; no longer SJ7.2, U1IO.PL_5C/7A/9A/12A/17A
- net N$2: now also SJ2.2, U4PWR.VCCIO1; no longer SJ3.2, U1PWR.VCCIO1
- net N$20: now also SJ7.2, U4IO.PL_5D/7B/9B/12B/17B; no longer SJ8.2, U1IO.PL_5D/7B/9B/12B/17B
- net N$3: now also SJ3.2, U4PWR.VCCIO2; no longer SJ2.2, U1PWR.VCCIO2
- net N$4: now also SJ4.2, U4PWR.VCCIO3; no longer SJ1.2, U1PWR.VCCIO3
- net N$5: now also R15.1, U1PB.PB8; no longer R15.2, U2PB.PB8
- net N$6: now also J4.7, R23.2; no longer J5.7, R12.2
- net N$7: now also R14.1, U1PB.PB0-ADC_IN8; no longer R14.2, U2PB.PB0-ADC_IN8
- net N$9: now also SJ8.2, U4IO.PB_4A/6C/9A/11A/13A; no longer SJ10.2, U1IO.PB_4A/6C/9A/11A/13A
- net N205481: now also C4.2, Q1.C1, R3.1; no longer C4.1, R2.1, X1.C1
- net N41567: now also D1.C; no longer D2.C
- net NRES: now also J4.10, U1CTL.NRST; no longer J5.10, U2CTL.NRST
- net OSC32_IN: now also U1PC.PC14-OSC32_IN; no longer U2PC.PC14-OSC32_IN
- net OSC32_OUT: now also U1PC.PC15-OSC32_OUT; no longer U2PC.PC15-OSC32_OUT
- net OSC_IN: now also C8.2; no longer C1.2
- net OSC_OUT: now also C9.2; no longer C11.2
- net PA7: now also D5.DIN, U1PA.PA7-ADC_IN7; no longer D1.DIN, U2PA.PA7-ADC_IN7
- net PB10: now also R12.1, U1PB.PB10; no longer R16.2, U2PB.PB10
- net PB11: now also R16.1, U1PB.PB11; no longer R17.1, U2PB.PB11
- net PF0: now also C7.2, Q1.C2, U1CTL.PF0-OSC_IN; no longer C5.2, U2CTL.PF0-OSC_IN, X1.C2
- net PF1: now also R3.2, U1CTL.PF1-OSC_OUT; no longer R2.2, U2CTL.PF1-OSC_OUT
- net PF4: now also R17.1, U1PDF.PF4; no longer R18.1, U2PDF.PF4
- net PF5: now also R11.1, U1PDF.PF5; no longer R19.1, U2PDF.PF5
- net PF6: now also R13.1, U1PDF.PF6; no longer R20.1, U2PDF.PF6
- net PF7: now also R18.1, R8.2, U1PDF.PF7; no longer R21.1, R22.2, U2PDF.PF7
- net PROGRAMN: now also U1PC.PC8, U4ERB.PROGRAMN/PT15D; no longer U1ERB.PROGRAMN/PT15D, U2PC.PC8
- net SN: now also U1PB.PB2, U4ERB.SN/PB20C; no longer U1ERB.SN/PB20C, U2PB.PB2
- net SWCLK: now also J4.4, R20.1, U1PA.PA14-SWCLK, U4ERB.TCK; no longer J5.4, R10.1, U1ERB.TCK, U2PA.PA14-SWCLK
- net SWDIO: now also J4.2, R19.2, U1PA.PA13-SWDIO, U4ERB.TMS; no longer J5.2, R9.2, U1ERB.TMS, U2PA.PA13-SWDIO
- net VBAT: now also U1PWR.VBAT; no longer U2PWR.VBAT
- net VCC-IN: now also D2.A, J1.VCC; no longer D5.A, J4.VCC
- net VCCIO: now also R8.1; no longer R22.1
- net VDDA: now also C10.1, C11.1, R5.1, U1PWR.VDDA; no longer C2.1, C3.1, R13.2, U2PWR.VDDA
- net VSSA: now also C10.2, C11.2, U1PWR.VSSA; no longer C2.2, C3.2, U2PWR.VSSA
Other:
- moved on the sheet: C1, C10, C11, C2, C3, C5, C6, C7, C8, C9, FB1, FB2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

Commit message: Renumbering & initial routing on Baselli
Parts:
- added X1, X2, X3, X4: M-BOLT-2, ELL-i-Connectors:M-BOLT-2
- C1: value 33n -> 22pF
- C2: value 1uF -> 22pF
- C3: value 100nF -> 33n
- C4: value 22pF -> 1uF
- C5: value 1uF -> 100nF
- C6: value 100nF -> 1uF
- C7: value 22pF -> 100nF
- R10: value 2K2 -> NP; device ELL-i-Passives:R0402 -> ELL-i-Passives:R0805
- R12, R16: value 0 -> 180
- R13, R14: value 180 -> 0
- R8: value NP -> 2K2; device ELL-i-Passives:R0805 -> ELL-i-Passives:R0402
Connections:
- removed net OSC_IN: C8.2, Y1.1
- removed net OSC_OUT: C9.2, Y1.2
- net +3V3: now also C4.1, C7.1, R8.1; no longer C2.1, C3.1, R10.1
- net +5V: now also OLPADS1.10
- net -RTS: now also C3.2; no longer C1.2
- net A4: now also R9.2; no longer R10.2
- net A5: now also R8.2; no longer R7.2
- net AREF: now also R5.1; no longer R5.2
- net D4: now also C3.1; no longer C1.1
- net D7: now also R11.1, SJ8.1; no longer R15.2, SJ10.1
- net D9: now also R12.1, SJ7.1; no longer R14.2, SJ12.1
- net DONE: now also SJ8.2; no longer SJ10.2
- net E0: now also R15.1, SJ9.1; no longer R17.2, SJ8.1
- net E1: now also R16.1, SJ10.1; no longer R11.2, SJ13.1
- net E12: now also R14.1, R7.2, SJ13.1; no longer R16.2, R9.2, SJ11.1
- net E13: now also R13.1, SJ14.1; no longer R12.2, SJ7.1
- net E2: now also R17.1, SJ11.1; no longer R13.2, SJ9.1
- net E3: now also R18.1, SJ12.1; no longer R18.2, SJ14.1
- net GNDI: now also C1.1, C2.1, C4.2, C7.2; no longer C2.2, C3.2, C4.1, C7.1
- net N$10: now also SJ10.2; no longer SJ13.2
- net N$12: now also SJ7.2; no longer SJ12.2
- net N$15: now also SJ11.2; no longer SJ9.2
- net N$16: now also SJ12.2; no longer SJ14.2
- net N$17: now also SJ13.2; no longer SJ11.2
- net N$20: now also SJ14.2; no longer SJ7.2
- net N$5: now also R11.2; no longer R15.1
- net N$7: now also R12.2; no longer R14.1
- net N$9: now also SJ9.2; no longer SJ8.2
- net N205481: now also C1.2; no longer C4.2
- net OSC32_IN: now also C8.2, Y1.2
- net OSC32_OUT: now also C9.2, Y1.1
- net PB10: now also R13.2; no longer R12.1
- net PB11: now also R14.2; no longer R16.1
- net PF0: now also C2.2; no longer C7.2
- net PF4: now also R15.2; no longer R17.1
- net PF5: now also R16.2; no longer R11.1
- net PF6: now also R17.2; no longer R13.1
- net PF7: now also R10.2, R18.2; no longer R18.1, R8.2
- net VCCIO: now also R10.1; no longer R8.1
- net VDDA: now also R5.2; no longer R5.1
Other:
- moved on the sheet: C1, C2, C3, C4, C5, C6, C7, R10, R11, R12, R13, R14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

Commit message: Mechanical design
Parts:
- added X5: POE-TP-PD-BELFUSE-T568A, ELL-i-Connectors:POE-TP-PD-BELFUSE-T568A
Changed lines of the file:
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@@
 <part name="X3" library="ELL-i-Connectors" deviceset="M-BOLT" device="-2"/>
 <part name="P+3" library="supply1" deviceset="+5V" device=""/>
+<part name="X5" library="ELL-i-Connectors" deviceset="POE-TP" device="-PD-BELFUSE-T568A"/>
 </parts>
 <sheets>
@@
 <instance part="X3" gate="M" x="139.7" y="220.98"/>
 <instance part="P+3" gate="1" x="-205.74" y="317.5"/>
+<instance part="X5" gate="G$1" x="-162.56" y="251.46"/>
 </instances>
 <busses>

Commit message: Remove excess punchdown connector from Baselli
Parts:
- removed X5: POE-TP-PD-BELFUSE-T568A, ELL-i-Connectors:POE-TP-PD-BELFUSE-T568A
Changed lines of the file:
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@@
 <part name="X3" library="ELL-i-Connectors" deviceset="M-BOLT" device="-2"/>
 <part name="P+3" library="supply1" deviceset="+5V" device=""/>
-<part name="X5" library="ELL-i-Connectors" deviceset="POE-TP" device="-PD-BELFUSE-T568A"/>
 </parts>
 <sheets>
@@
 <instance part="X3" gate="M" x="139.7" y="220.98"/>
 <instance part="P+3" gate="1" x="-205.74" y="317.5"/>
-<instance part="X5" gate="G$1" x="-162.56" y="251.46"/>
 </instances>
 <busses>

Commit message: Preliminary work on Baselli
Parts:
- added C12: 100nF, ELL-i-Passives:C0402
- added C13: 1uF, ELL-i-Passives:C0402
- D3: value BAT60J -> DIODE-SCHOTTKY-BAT60J; device ell-i:BAT60J -> SparkFun-DiscreteSemi:DIODE-SCHOTTKY-BAT60J
- R10, R11, R12, R13, R14, R15, R16, R17, R18, R23, R5: device ELL-i-Passives:R0805 -> ELL-i-Passives:R0603
Connections:
- net +3V3: now also C12.1, C13.1
- net GNDI: now also C12.2, C13.2
