File: Baselli/Baselli.brd (EAGLE design)
At the start: 54 x 54 mm, 73 parts, among them J2 DF12-ELLI-HEADER-TOP, J3 DF12-ELLI-RECEPTABLE-BOTTOM, J4 FTDI-SER-6-PP, J5 JTAG_PROG, Q1 IRLML2244, SW1 A6H-2101, U1 LCMXO2-256HC-4SG32, U2 STM32F051R, X1 8MHz NP

Commit message: Add 32 kHz oscillator to .brd & rename
Parts:
- added C1, C11: 15 pF, ELL-i-Passives:C0402
- added X2: 32.768 kHz, SparkFun-FreqCtrl:CRYSTAL-32KHZ-SMD
Connections:
- new net OSC_IN: C1.2, X2.X1
- new net OSC_OUT: C11.2, X2.X2
- net GNDI: now also C1.1, C11.1
Changed lines of the file:
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@@
 <element name="R15" library="ELL-i-Passives" package="R0805" value="180" x="14" y="39"/>
 <element name="R14" library="ELL-i-Passives" package="R0805" value="180" x="14" y="43"/>
+<element name="C1" library="ELL-i-Passives" package="C0402" value="15 pF" x="4" y="7"/>
+<element name="C11" library="ELL-i-Passives" package="C0402" value="15 pF" x="10" y="4"/>
+<element name="X2" library="SparkFun-FreqCtrl" package="CRYSTAL-32KHZ-SMD" value="32.768 kHz" x="-9" y="-4">
+<attribute name="PROD_ID" value="XTAL-07894" x="-9" y="-4" size="1.778" layer="27" display="off"/>
+</element>
 </elements>
 <signals>
@@
 <contactref element="SJ6" pad="1"/>
 <contactref element="D1" pad="3"/>
+<contactref element="C1" pad="1"/>
+<contactref element="C11" pad="1"/>
 <wire x1="43.58" y1="37.66" x2="50.38" y2="37.66" width="0" layer="19" extent="1-1"/>
 <wire x1="51.56" y1="29.49" x2="50.38" y2="37.66" width="0" layer="19" extent="1-1"/>
@@
 <wire x1="23.75" y1="32.75" x2="30.035" y2="37.33" width="0" layer="19" extent="1-1"/>
 <wire x1="12.45" y1="11" x2="26.25" y2="13.5" width="0" layer="19" extent="1-16"/>
+<wire x1="9.525" y1="4" x2="12.45" y2="11" width="0" layer="19" extent="1-16"/>
+<wire x1="3.525" y1="7" x2="9.525" y2="4" width="0" layer="19" extent="1-1"/>
 <wire x1="3.1999" y1="22.25" x2="12.45" y2="11" width="0" layer="19" extent="16-16"/>
 <wire x1="3.1999" y1="22.25" x2="3.1999" y2="22.25" width="0" layer="19" extent="1-16"/>
@@
 <contactref element="R3" pad="2"/>
 <contactref element="SW1" pad="4"/>
-<wire x1="48.645" y1="20.41" x2="43.265" y2="25.68" width="0" layer="19" extent="1-1"/>
-<wire x1="51.56" y1="21.87" x2="48.645" y2="20.41" width="0" layer="19" extent="1-1"/>
+<wire x1="48.645" y1="20.41" x2="51.56" y2="21.87" width="0" layer="19" extent="1-1"/>
+<wire x1="43.265" y1="25.68" x2="48.645" y2="20.41" width="0" layer="19" extent="1-1"/>
 </signal>
 <signal name="JTAGEN_GATE">
@@
 <contactref element="Q1" pad="1"/>
 <wire x1="39.865" y1="20.41" x2="45.67" y2="21.47" width="0" layer="19" extent="1-1"/>
-<wire x1="41.39" y1="14.8271" x2="45.67" y2="21.47" width="0" layer="19" extent="1-1"/>
+<wire x1="41.39" y1="14.8271" x2="39.865" y2="20.41" width="0" layer="19" extent="1-1"/>
 </signal>
 <signal name="PF6">
@@
 <wire x1="0.56" y1="22.87" x2="32.75" y2="23.25" width="0" layer="19" extent="1-1"/>
 </signal>
+<signal name="OSC_IN">
+<contactref element="C1" pad="2"/>
+<contactref element="X2" pad="X1"/>
+<wire x1="4.475" y1="7" x2="-7.73" y2="-4" width="0" layer="19" extent="1-1"/>
+</signal>
+<signal name="OSC_OUT">
+<contactref element="C11" pad="2"/>
+<contactref element="X2" pad="X2"/>
+<wire x1="-10.27" y1="-4" x2="10.475" y2="4" width="0" layer="19" extent="1-1"/>
+</signal>
 </signals>

Commit message: Fixups and renumbering in Baselli
Parts:
- removed J5: JTAG_PROG, ELL-i-Connectors:CLP-105-02-X-D
- removed U2: STM32F051R, ELL-i-DigitalIC:LQFP64
- removed X1: 8MHz NP, SparkFun-FreqCtrl:CRYSTAL-SMD-3225-GND
- added J1: FTDI-SER-6-PP, ELL-i-Connectors:FTDI-SER-6-SIL
- added Q2: IRLML2244, SparkFun-DiscreteSemi:SOT23-3
- added U4: LCMXO2-256HC-4SG32, ELL-i-DigitalIC:QFN-32
- C1: value 15 pF -> 33n
- C10: value 33n -> 1uF
- C11: value 15 pF -> 10nF
- C3: value 10nF -> 100nF
- C5: value 22pF -> 1uF
- C7: value 1uF -> 22pF
- C8: value 1uF -> 15 pF
- C9: value 100nF -> 15 pF
- D1: value WS2182B -> GREEN; device SparkFun-LED:WS2812B -> SparkFun-LED:LED-0603
- D2: value GREEN -> BAT60J; device SparkFun-LED:LED-0603 -> SparkFun-DiscreteSemi:SOD-323
- D5: value BAT60J -> WS2182B; device SparkFun-DiscreteSemi:SOD-323 -> SparkFun-LED:WS2812B
- J4: value FTDI-SER-6-PP -> JTAG_PROG; device ELL-i-Connectors:FTDI-SER-6-SIL -> ELL-i-Connectors:CLP-105-02-X-D
- Q1: value IRLML2244 -> 8MHz NP; device SparkFun-DiscreteSemi:SOT23-3 -> SparkFun-FreqCtrl:CRYSTAL-SMD-3225-GND
- R10: value 4K7 (NP) -> 2K2; device ELL-i-Passives:R0603 -> ELL-i-Passives:R0402
- R11: value 47K -> 180; device ELL-i-Passives:R0402 -> ELL-i-Passives:R0805
- R12: value NP -> 0
- R13: value 10k -> 180
- R17: value 0 -> 180
- R19, R21: value 180 -> 10K; device ELL-i-Passives:R0805 -> ELL-i-Passives:R0402
- R2: value 390R -> 10k
- R20: value 180 -> 4K7 (NP); device ELL-i-Passives:R0805 -> ELL-i-Passives:R0603
- R22: value NP -> 47K; device ELL-i-Passives:R0805 -> ELL-i-Passives:R0402
- R23: value 1k5 -> NP; device ELL-i-Passives:R0402 -> ELL-i-Passives:R0805
- R3: value 10k -> 390R
- R4: value 2K2 -> 1k5
- R5: value 2K2 -> 10k; device ELL-i-Passives:R0402 -> ELL-i-Passives:R0805
- R8: value 10K -> NP; device ELL-i-Passives:R0402 -> ELL-i-Passives:R0805
- R9: value 10K -> 2K2
- U1: value LCMXO2-256HC-4SG32 -> STM32F051R; device ELL-i-DigitalIC:QFN-32 -> ELL-i-DigitalIC:LQFP64
- moved D2 45.7 mm to (47.8, 23.6), turned to 0 degrees
- moved C1 45.0 mm to (47.8, 17.4)
- moved C11 41.7 mm to (26.5, 42.3)
- moved C8 41.5 mm to (4.00, 7.00)
- moved R12 40.3 mm to (14.0, 39.0)
- moved C9 39.7 mm to (10.0, 4.00)
- moved R11 34.0 mm to (14.0, 43.0)
- moved D1 32.9 mm to (5.17, 40.0), turned to 90 degrees
- moved C10 31.6 mm to (26.0, 40.3)
- moved R8 29.7 mm to (14.0, 11.0)
- moved R20 28.8 mm to (29.7, 43.2), turned to 90 degrees
- moved R4 28.7 mm to (35.1, 21.6)
- moved R21 28.5 mm to (41.5, 22.4)
- moved R22 27.1 mm to (39.4, 20.4)
- moved D5 23.3 mm to (37.7, 44.6), turned to 180 degrees
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- renumbered X2 to Y1
Connections:
- net +3V3: now also C2.1, C3.1, C5.1, D1.A, D2.C, J4.1, Q2.2, R10.1, R19.1, R22.1, U1.32, U1.64, U4.18, U4.2; no longer C7.1, C8.1, C9.1, D2.A, D5.C, J5.1, Q1.2, R11.1, R4.1, R5.1, U1.18, U1.2, U2.32, U2.64
- net +5V: now also D5.1; no longer D1.1
- net -RTS: now also C1.2; no longer C10.2
- net A0: now also U1.14; no longer U2.14
- net A1: now also U1.16; no longer U2.16
- net A2: now also U1.20; no longer U2.20
- net A3: now also U1.21; no longer U2.21
- net A4: now also R10.2, U1.62, U4.27; no longer R7.2, U1.27, U2.62
- net A5: now also R7.2, U1.58, U4.28; no longer R6.2, U1.28, U2.58
- net AREF: now also R5.2; no longer R13.1
- net BOOT0: now also R4.2, U1.60; no longer R23.2, U2.60
- net BOOT0TX: now also J1.TXD, R2.1; no longer J4.TXD, R3.2
- net CSSPIN: now also U1.53, U4.8; no longer U1.8, U2.53
- net D0: now also R2.2, U1.43; no longer R3.1, U2.43
- net D1: now also J1.RXD, U1.42; no longer J4.RXD, U2.42
- net D10: now also J4.6, U1.50, U4.1; no longer J5.6, U1.1, U2.50
- net D11: now also U1.57, U4.17; no longer U1.17, U2.57
- net D12: now also U1.22, U4.10; no longer U1.10, U2.22
- net D13: now also U1.55, U4.9; no longer U1.9, U2.55
- net D2: now also U1.54; no longer U2.54
- net D3: now also J1.-CTS, U1.44; no longer J4.-CTS, U2.44
- net D4: now also C1.1, J1.-RTS, U1.45; no longer C10.1, J4.-RTS, U2.45
- net D5: now also U1.27; no longer U2.27
- net D6: now also U1.17; no longer U2.17
- net D7: now also R15.2, SJ10.1; no longer R15.1, SJ14.1
- net D8: now also U1.59; no longer U2.59
- net D9: now also R14.2, SJ12.1; no longer R14.1, SJ9.1
- net DONE: now also SJ10.2, U4.23; no longer SJ14.2, U1.23
- net DOUT: now also D5.2; no longer D1.2
- net E0: now also R17.2, SJ8.1; no longer R18.2, SJ10.1
- net E1: now also R11.2, SJ13.1; no longer R19.2, SJ11.1
- net E10: now also U1.37; no longer U2.37
- net E11: now also U1.38; no longer U2.38
- net E12: now also R16.2, R9.2, SJ11.1; no longer R17.2, R5.2, SJ7.1
- net E13: now also R12.2, R6.2, SJ7.1; no longer R16.1, R4.2, SJ8.1
- net E14: now also U1.33; no longer U2.33
- net E15: now also U1.36; no longer U2.36
- net E16: now also U1.35; no longer U2.35
- net E17: now also U1.34; no longer U2.34
- net E18: now also U1.52; no longer U2.52
- net E19: now also U1.51; no longer U2.51
- net E2: now also R13.2, SJ9.1; no longer R20.2, SJ12.1
- net E3: now also R18.2, SJ14.1; no longer R21.2, SJ13.1
- net E4: now also U1.8; no longer U2.8
- net E5: now also U1.9; no longer U2.9
- net E6: now also U1.10; no longer U2.10
- net E7: now also U1.11; no longer U2.11
- net E8: now also U1.24; no longer U2.24
- net E9: now also U1.25; no longer U2.25
- net ETH_INT: now also U1.15; no longer U2.15
- net ETH_SS: now also U1.2; no longer U2.2
- net GNDI: now also C2.2, C3.2, C4.1, C5.2, C7.1, C8.1, C9.1, D5.3, J1.GND, J4.5, J4.9, Q1.2, Q1.4, R20.2, R21.1, R4.1, U1.31, U1.63, U4.22, U4.3; no longer C1.1, C11.1, C4.2, C5.1, C7.2, C8.2, C9.2, D1.3, J4.GND, J5.5, J5.9, R10.2, R12.1, R8.1, U1.22, U1.3, U2.31, U2.63, X1.2, X1.4
- net JTAGENB: now also Q2.3, R21.2, U4.26; no longer Q1.3, R8.2, U1.26
- net JTAGENB_MCU: now also U1.56; no longer U2.56
- net JTAGEN_GATE: now also J4.3, Q2.1, R22.2; no longer J5.3, Q1.1, R11.2
- net JTDI: now also J4.8, U1.40, U4.32; no longer J5.8, U1.32, U2.40
- net MCO: now also U1.41, U4.21; no longer U1.21, U2.41
- net N$1: now also SJ1.2, U4.24, U4.31; no longer SJ4.2, U1.24, U1.31
- net N$10: now also SJ13.2, U4.12; no longer SJ11.2, U1.12
- net N$12: now also SJ12.2, U4.20; no longer SJ9.2, U1.20
- net N$15: now also SJ9.2, U4.13; no longer SJ12.2, U1.13
- net N$16: now also SJ14.2, U4.14; no longer SJ13.2, U1.14
- net N$17: now also SJ11.2, U4.4; no longer SJ7.2, U1.4
- net N$2: now also SJ2.2, U4.19; no longer SJ3.2, U1.19
- net N$20: now also SJ7.2, U4.5; no longer SJ8.2, U1.5
- net N$3: now also SJ3.2, U4.15, U4.7; no longer SJ2.2, U1.15, U1.7
- net N$4: now also SJ4.2, U4.6; no longer SJ1.2, U1.6
- net N$5: now also R15.1, U1.61; no longer R15.2, U2.61
- net N$6: now also J4.7, R23.2; no longer J5.7, R12.2
- net N$7: now also R14.1, U1.26; no longer R14.2, U2.26
- net N$9: now also SJ8.2, U4.11; no longer SJ10.2, U1.11
- net N205481: now also C4.2, Q1.1, R3.1; no longer C4.1, R2.1, X1.1
- net N41567: now also D1.C; no longer D2.C
- net NRES: now also J4.10, U1.7; no longer J5.10, U2.7
- net OSC32_IN: now also U1.3; no longer U2.3
- net OSC32_OUT: now also U1.4; no longer U2.4
- net OSC_IN: now also C8.2; no longer C1.2
- net OSC_OUT: now also C9.2; no longer C11.2
- net PA7: now also D5.4, U1.23; no longer D1.4, U2.23
- net PB10: now also R12.1, U1.29; no longer R16.2, U2.29
- net PB11: now also R16.1, U1.30; no longer R17.1, U2.30
- net PF0: now also C7.2, Q1.3, U1.5; no longer C5.2, U2.5, X1.3
- net PF1: now also R3.2, U1.6; no longer R2.2, U2.6
- net PF4: now also R17.1, U1.18; no longer R18.1, U2.18
- net PF5: now also R11.1, U1.19; no longer R19.1, U2.19
- net PF6: now also R13.1, U1.47; no longer R20.1, U2.47
- net PF7: now also R18.1, R8.2, U1.48; no longer R21.1, R22.2, U2.48
- net PROGRAMN: now also U1.39, U4.25; no longer U1.25, U2.39
- net SN: now also U1.28, U4.16; no longer U1.16, U2.28
- net SWCLK: now also J4.4, R20.1, U1.49, U4.30; no longer J5.4, R10.1, U1.30, U2.49
- net SWDIO: now also J4.2, R19.2, U1.46, U4.29; no longer J5.2, R9.2, U1.29, U2.46
- net VBAT: now also U1.1; no longer U2.1
- net VCC-IN: now also D2.A, J1.VCC; no longer D5.A, J4.VCC
- net VCCIO: now also R8.1; no longer R22.1
- net VDDA: now also C10.1, C11.1, R5.1, U1.13; no longer C2.1, C3.1, R13.2, U2.13
- net VSSA: now also C10.2, C11.2, U1.12; no longer C2.2, C3.2, U2.12

Commit message: Renumbering & initial routing on Baselli
Parts:
- added X1, X2, X3, X4: M-BOLT-2, ELL-i-Connectors:M2-1
- C1: value 33n -> 22pF
- C2: value 1uF -> 22pF
- C3: value 100nF -> 33n
- C4: value 22pF -> 1uF
- C5: value 1uF -> 100nF
- C6: value 100nF -> 1uF
- C7: value 22pF -> 100nF
- R10: value 2K2 -> NP; device ELL-i-Passives:R0402 -> ELL-i-Passives:R0805
- R12, R16: value 0 -> 180
- R13, R14: value 180 -> 0
- R8: value NP -> 2K2; device ELL-i-Passives:R0805 -> ELL-i-Passives:R0402
- moved TP4 40.7 mm to (41.0, 5.00), turned to 270 degrees
- moved D3 38.6 mm to (37.0, 36.0), turned to 90 degrees
- moved Y1 38.5 mm to (25.0, 14.0), turned to 270 degrees
- moved TP2 34.3 mm to (51.0, 37.0)
- moved R23 31.1 mm to (12.5, 10.0), turned to 90 degrees
- moved C3 30.5 mm to (46.0, 21.0), turned to 90 degrees
- moved Q2 28.3 mm to (16.4, 20.8), turned to 0 degrees
- moved C2 25.9 mm to (23.5, 17.5)
- moved J4 25.9 mm to (17.0, 13.0), turned to 270 degrees
- moved SJ11 24.7 mm to (23.0, 30.0)
- moved SJ13 23.8 mm to (20.0, 30.0)
- moved SJ15 23.3 mm to (16.0, 30.0)
- moved R22 22.9 mm to (16.6, 17.9), turned to 90 degrees
- moved C8 22.9 mm to (22.5, 20.5), turned to 90 degrees
- moved C9 21.3 mm to (23.5, 20.5), turned to 90 degrees
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Connections:
- removed net OSC_IN: C8.2, Y1.X1
- removed net OSC_OUT: C9.2, Y1.X2
- net +3V3: now also C4.1, C7.1, R8.1; no longer C2.1, C3.1, R10.1
- net +5V: now also OLPADS1.10
- net -RTS: now also C3.2; no longer C1.2
- net A4: now also R9.2; no longer R10.2
- net A5: now also R8.2; no longer R7.2
- net AREF: now also R5.1; no longer R5.2
- net D4: now also C3.1; no longer C1.1
- net D7: now also R11.1, SJ8.1; no longer R15.2, SJ10.1
- net D9: now also R12.1, SJ7.1; no longer R14.2, SJ12.1
- net DONE: now also SJ8.2; no longer SJ10.2
- net E0: now also R15.1, SJ9.1; no longer R17.2, SJ8.1
- net E1: now also R16.1, SJ10.1; no longer R11.2, SJ13.1
- net E12: now also R14.1, R7.2, SJ13.1; no longer R16.2, R9.2, SJ11.1
- net E13: now also R13.1, SJ14.1; no longer R12.2, SJ7.1
- net E2: now also R17.1, SJ11.1; no longer R13.2, SJ9.1
- net E3: now also R18.1, SJ12.1; no longer R18.2, SJ14.1
- net GNDI: now also C1.1, C2.1, C4.2, C7.2; no longer C2.2, C3.2, C4.1, C7.1
- net N$10: now also SJ10.2; no longer SJ13.2
- net N$12: now also SJ7.2; no longer SJ12.2
- net N$15: now also SJ11.2; no longer SJ9.2
- net N$16: now also SJ12.2; no longer SJ14.2
- net N$17: now also SJ13.2; no longer SJ11.2
- net N$20: now also SJ14.2; no longer SJ7.2
- net N$5: now also R11.2; no longer R15.1
- net N$7: now also R12.2; no longer R14.1
- net N$9: now also SJ9.2; no longer SJ8.2
- net N205481: now also C1.2; no longer C4.2
- net OSC32_IN: now also C8.2, Y1.X2
- net OSC32_OUT: now also C9.2, Y1.X1
- net PB10: now also R13.2; no longer R12.1
- net PB11: now also R14.2; no longer R16.1
- net PF0: now also C2.2; no longer C7.2
- net PF4: now also R15.2; no longer R17.1
- net PF5: now also R16.2; no longer R11.1
- net PF6: now also R17.2; no longer R13.1
- net PF7: now also R10.2, R18.2; no longer R18.1, R8.2
- net VCCIO: now also R10.1; no longer R8.1
- net VDDA: now also R5.2; no longer R5.1
Routing:
- net +5V: track 0.00 -> 56.2 mm
- net +3V3: track 0.00 -> 46.6 mm
- net GNDI: track 0.00 -> 35.7 mm
- net VCCIO: track 0.00 -> 21.5 mm
- net NRES: track 0.00 -> 14.3 mm
- net E1: track 0.00 -> 12.6 mm, vias 0 -> 2
- net DOUT: track 0.00 -> 12.5 mm
- net E12: track 0.00 -> 11.7 mm
- net E0: track 0.00 -> 11.5 mm
- net SWCLK: track 0.00 -> 10.6 mm
- net BOOT0TX: track 0.00 -> 9.90 mm
- net VBATT: track 0.00 -> 9.08 mm
- net JTAGEN_GATE: track 0.00 -> 9.00 mm
- net -RTS: track 0.00 -> 8.73 mm
- net E13: track 0.00 -> 6.62 mm
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
Commit message: Mechanical design
Parts:
- added X5: POE-TP-PD-BELFUSE-T568A, ELL-i-Connectors:BELFUSE-SS-51-PD-T568A
- moved D1 7.00 mm to (6.00, 44.5)
- moved R1 5.10 mm to (4.00, 42.5)
- moved X1 2.12 mm to (5.50, 39.5)
- moved X2 2.12 mm to (48.5, 39.5)
- moved X3 2.12 mm to (5.50, 14.5)
- moved X4 2.12 mm to (48.5, 14.5)
- moved TP2 1.00 mm to (52.0, 37.0)
- moved TP3 1.00 mm to (52.0, 17.0)
Connections:
- new net POE+: X5.4, X5.5
- new net POE-: X5.7, X5.8
Routing:
- net +3V3: track 46.6 -> 51.5 mm
- net GNDI: track 35.7 -> 39.9 mm
Changed lines of the file:
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@@
 <element name="C4" library="ELL-i-Passives" package="C0402" value="1uF" x="32.87" y="38.41"/>
 <element name="C5" library="ELL-i-Passives" package="C0402" value="100nF" x="33.33" y="37.41"/>
-<element name="D1" library="SparkFun-LED" package="LED-0603" value="GREEN" x="6" y="37.5" rot="R90">
-<attribute name="PROD_ID" value="DIO-00821" x="106.33" y="117.51" size="1.778" layer="27" rot="R90" display="off"/>
+<element name="D1" library="SparkFun-LED" package="LED-0603" value="GREEN" x="6" y="44.5" rot="R90">
+<attribute name="PROD_ID" value="DIO-00821" x="106.33" y="124.51" size="1.778" layer="27" rot="R90" display="off"/>
 </element>
-<element name="R1" library="ELL-i-Passives" package="R0402" value="150R" x="3" y="37.5" rot="R180"/>
+<element name="R1" library="ELL-i-Passives" package="R0402" value="150R" x="4" y="42.5" rot="R180"/>
 <element name="R3" library="ELL-i-Passives" package="R0402" value="390R" x="30" y="19"/>
 <element name="R7" library="ELL-i-Passives" package="R0402" value="2K2" x="9" y="34" rot="R180"/>
@@
 <element name="D2" library="SparkFun-DiscreteSemi" package="SOD-323" value="BAT60J" x="46" y="28"/>
 <element name="Q1" library="SparkFun-FreqCtrl" package="CRYSTAL-SMD-3225-GND" value="8MHz NP" x="27" y="18" rot="R180"/>
-<element name="TP2" library="ELL-i-Passives" package="TP_5021" value="" x="51" y="37"/>
-<element name="TP3" library="ELL-i-Passives" package="TP_5021" value="" x="51" y="17"/>
+<element name="TP2" library="ELL-i-Passives" package="TP_5021" value="" x="52" y="37"/>
+<element name="TP3" library="ELL-i-Passives" package="TP_5021" value="" x="52" y="17"/>
 <element name="TP4" library="ELL-i-Passives" package="TP_5021" value="" x="41" y="5" rot="R270"/>
 <element name="TP5" library="ELL-i-Passives" package="TP_5021" value="" x="13" y="5" rot="R90"/>
@@
 <attribute name="PROD_ID" value="XTAL-07894" x="25" y="14" size="1.778" layer="27" rot="R270" display="off"/>
 </element>
-<element name="X1" library="ELL-i-Connectors" package="M2-1" value="M-BOLT-2" x="7" y="41"/>
-<element name="X2" library="ELL-i-Connectors" package="M2-1" value="M-BOLT-2" x="47" y="41"/>
-<element name="X4" library="ELL-i-Connectors" package="M2-1" value="M-BOLT-2" x="47" y="13"/>
-<element name="X3" library="ELL-i-Connectors" package="M2-1" value="M-BOLT-2" x="7" y="13"/>
+<element name="X1" library="ELL-i-Connectors" package="M2-1" value="M-BOLT-2" x="5.5" y="39.5"/>
+<element name="X2" library="ELL-i-Connectors" package="M2-1" value="M-BOLT-2" x="48.5" y="39.5"/>
+<element name="X4" library="ELL-i-Connectors" package="M2-1" value="M-BOLT-2" x="48.5" y="14.5"/>
+<element name="X3" library="ELL-i-Connectors" package="M2-1" value="M-BOLT-2" x="5.5" y="14.5"/>
+<element name="X5" library="ELL-i-Connectors" package="BELFUSE-SS-51-PD-T568A" value="POE-TP-PD-BELFUSE-T568A" x="27" y="45" rot="R180"/>
 </elements>
 <signals>
@@
 <contactref element="D1" pad="C"/>
 <contactref element="R1" pad="1"/>
-<wire x1="3.475" y1="37.5" x2="5.123" y2="37.5" width="0.254" layer="1"/>
+<wire x1="4.475" y1="42.5" x2="5.123" y2="44.5" width="0.254" layer="1"/>
 </signal>
 <signal name="VSSA">
@@
 <wire x1="8.525" y1="36.5" x2="8.189125" y2="37.310875" width="0.254" layer="1" curve="45"/>
 <wire x1="8.189125" y1="37.310875" x2="8" y2="37.5" width="0.254" layer="1"/>
-<wire x1="8" y1="37.5" x2="6.877" y2="37.5" width="0.254" layer="1"/>
+<wire x1="8" y1="37.5" x2="6.877" y2="44.5" width="0.254" layer="1"/>
 <wire x1="19" y1="7.8128" x2="24" y2="7.8128" width="0.254" layer="16"/>
 <wire x1="24" y1="7.8128" x2="29" y2="7.8128" width="0.254" layer="16"/>
@@
 <wire x1="8.525" y1="36.5" x2="9.475" y2="34" width="0" layer="19" extent="1-1"/>
 <wire x1="29" y1="7.8128" x2="34" y2="7.8128" width="0.254" layer="16"/>
-<wire x1="51" y1="17" x2="52" y2="17" width="0.254" layer="1"/>
 <wire x1="52" y1="17" x2="53" y2="18" width="0.254" layer="1"/>
 <wire x1="53" y1="18" x2="53" y2="29" width="0.254" layer="1"/>
@@
 <wire x1="1.25" y1="30.75" x2="1" y2="31" width="0.254" layer="1" curve="-90"/>
 <wire x1="1" y1="31" x2="1" y2="37.5" width="0.254" layer="1"/>
-<wire x1="1" y1="37.5" x2="2.525" y2="37.5" width="0.254" layer="1"/>
+<wire x1="1" y1="37.5" x2="3.525" y2="42.5" width="0.254" layer="1"/>
 <wire x1="33.885" y1="36.41" x2="43.475" y2="33" width="0" layer="19" extent="1-1"/>
 <wire x1="33.805" y1="37.41" x2="33.885" y2="36.41" width="0" layer="19" extent="1-1"/>
@@
 <wire x1="51" y1="33.35" x2="43.825" y2="33.35" width="0.254" layer="1"/>
 <wire x1="43.825" y1="33.35" x2="43.475" y2="33" width="0.254" layer="1" curve="90"/>
-<wire x1="51" y1="37" x2="51" y2="33.35" width="0.254" layer="1"/>
+<wire x1="52" y1="37" x2="51" y2="33.35" width="0.254" layer="1"/>
 <wire x1="15.3871" y1="10.46" x2="16.46" y2="10.46" width="0.254" layer="1"/>
 <wire x1="16.46" y1="10.46" x2="17" y2="11" width="0.254" layer="1"/>
@@
 <wire x1="12.1" y1="16" x2="23.25" y2="23.25" width="0" layer="19" extent="1-1"/>
 </signal>
+<signal name="POE+">
+<contactref element="X5" pad="4"/>
+<contactref element="X5" pad="5"/>
+<wire x1="13.792" y1="45" x2="10.49" y2="45" width="0" layer="19" extent="1-1"/>
+</signal>
+<signal name="POE-">
+<contactref element="X5" pad="7"/>
+<contactref element="X5" pad="8"/>
+<wire x1="40.208" y1="45" x2="43.51" y2="45" width="0" layer="19" extent="1-1"/>
+</signal>
 </signals>
