File: Arduelli/Arduelli.sch (EAGLE design)
At the start: 86 parts, among them J1 47346-0001, J2 DF12-ELLI-RECEPTABLE-BOTTOM, J4 FTDI-SER-6-PP, J5 JTAG_PROG, J6 47346-0001, Q1 NTZD3152P, Q2 2N7002PT, Q3 MOSFET-PCHANNELIRLML2244, U1 ARDUINO_SHIELDLONGPADS, U2 STM32F103RBT, U3 ADUM4160BRWZ, U4 ADUM4160BRWZ, U5 NCP1117, X1 M-BOLT-2, X2 M-BOLT-2, X3 M-BOLT-2, X4 M-BOLT-2, X5 M-BOLT-2, Y1 8MHz

Commit message: Added JTAG power logic+Modified Power Arbiter gnds
Parts:
- added C13: 0.1uF, ELL-i-Passives:C0402
- added R26: 4k7, ELL-i-Passives:R0402
- added R27: 10k, ELL-i-Passives:R0402
- added SJ1, SJ2: OPEN, SparkFun-Passives:SOLDERJUMPERNO
- added TP1, TP5, TP6: TEST_POINT-5000, ELL-i-Passives:TEST_POINT-5000
- D3: device tinycircuits:AS-ITM-00111 -> ELL-i-DiscreteSemi:DIODE-SCHOTTKYB2100
- Q2: device tinycircuits:AS-ITM-00110 -> ELL-i-DiscreteSemi:2N7002PT
Connections:
- removed net N$31: U2PB.PB0-ADC_IN8
- removed net USB_POWER: Q1.D1, R1.2
- removed net VCC: C1.1, Q1.S1, Q1.S2, R2.2
- new net N$15: TP1.P$1, U2PB.PB3
- new net TPWR_DETECT: C13.1, R26.1, R27.2, U2PB.PB0-ADC_IN8
- net +3V3: now also C1.1, D3.A, Q1.D1, Q1.G1, Q1.S1, Q1.S2, Q2.G, R1.2, R2.2, R3.2, SJ2.2
- net +5V: no longer D3.A, Q1.G1, Q2.G, R3.2
- net AGND: now also C1.2, C13.2, R27.1
- net D3: now also SJ4.1
- net D4: now also SJ1.1, SJ2.1; no longer SJ4.1
- net GND: no longer C1.2, Q2.S, R1.1
- net GNDA: now also Q2.S
- net GNDI: now also R1.1
- net HDD+: no longer SJ4.2
- net HDD-: no longer SJ3.2
- net LDO_GND: now also SJ1.2, SJ4.2
- net LDO_IN: now also SJ3.2
- net RX: now also TP5.P$1
- net TPWR: now also R26.2
- net TX: now also TP6.P$1
Other:
- note added: "VCC of Arduelli"
- note removed: "UGND"
- note removed: "VCC of Ardueli"
- note removed: "V_USB"
- moved on the sheet: SJ3, SJ4
