File: Arduelli/Arduelli.brd (EAGLE design)
At the start: 100 x 80 mm, 94 parts, among them J1 47346-0001, J2 DF12-ELLI-RECEPTABLE-BOTTOM, J4 FTDI-SER-6-PP, J5 JTAG_PROG, J6 47346-0001, Q1 NTZD3152P, Q2 2N7002PT, Q3 MOSFET-PCHANNELIRLML2244, U1 ARDUINO_SHIELDLONGPADS, U2 STM32F103RBT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

Commit message: Preliminary version of Arduelli board - 2
Parts:
- moved R12 165.4 mm to (38.1, 11.4)
- moved S2 163.4 mm to (77.5, 49.5)
- moved U5 162.9 mm to (66.0, 50.8)
- moved J5 161.1 mm to (67.3, 59.7)
- moved D9 155.3 mm to (45.7, 57.1)
- moved D2 152.2 mm to (15.2, 20.3)
- moved R11 151.1 mm to (19.1, 10.2)
- moved D8 150.3 mm to (45.7, 61.0)
- moved SW1 150.2 mm to (74.9, 36.8)
- moved SW3 147.8 mm to (67.3, 36.8)
- moved R6 147.6 mm to (19.1, 6.35)
- moved FB3 146.2 mm to (69.8, 74.9)
- moved R4 141.7 mm to (17.8, 8.89)
- moved R9 136.7 mm to (12.7, 21.6)
- moved FB1 124.0 mm to (11.4, 16.5)
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
Commit message: Preliminary version of Arduelli board - 3
Parts:
- moved R16 200.6 mm to (99.1, 68.6)
- moved R20 186.8 mm to (77.5, 69.8)
- moved R15 181.5 mm to (81.3, 67.3)
- moved R17 178.7 mm to (72.4, 64.8)
- moved R14 174.7 mm to (76.2, 66.0)
- moved SJ16 170.6 mm to (61.0, 45.7)
- moved SJ2 170.3 mm to (61.0, 63.5)
- moved R18 169.8 mm to (64.8, 78.7)
- moved R7 162.6 mm to (43.2, 10.2)
- moved R8 162.5 mm to (38.1, 7.62)
- moved SJ1 151.1 mm to (45.7, 71.1)
- moved TP3 149.1 mm to (48.3, 41.9)
- moved C16 147.2 mm to (40.6, 36.8)
- moved Y1 144.5 mm to (38.1, 48.3)
- moved SJ6 141.4 mm to (45.7, 67.3)
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